File: pcb/rp2040-board.kicad_pcb (KiCad board)
At the start: 4 copper layers, 52 parts, among them J1 DMX, J1 RS485, J2 GPIO, J3 ELRS, J4 OLED, J5 Conn_ARM_JTAG_SWD_10, J6 USB_C_Receptacle_USB2.0_16P, SW1 USB Boot, SW2 RotaryEncoder_Switch, SW3 Reset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

Commit message: pcb wip
Parts:
- moved C1 80.2 mm to (132.6, 114.9)
- moved C2 80.2 mm to (132.6, 116.8)
- moved C5 63.5 mm to (143.2, 100.6), turned to 180 degrees
- moved C6 62.8 mm to (143.2, 97.0), turned to 180 degrees
- moved R2 50.2 mm to (127.5, 116.8)
- moved R1 50.2 mm to (127.5, 114.8)
- moved R5 30.4 mm to (143.2, 98.2)
- moved SW3 29.6 mm to (111.8, 137.2)
- moved R4 26.6 mm to (143.2, 99.4)
- moved U1 25.4 mm to (139.7, 110.6), turned to 90 degrees
- moved SW1 25.4 mm to (96.5, 127.0)
- moved J5 14.4 mm to (164.5, 113.0)
- moved Y1 12.0 mm to (147.5, 122.8)
- moved R7 12.0 mm to (148.1, 128.7)
- moved C16 12.0 mm to (151.9, 125.5)
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
Commit message: pcb wip
Parts:
- moved C13 68.8 mm to (147.0, 106.0), turned to -90 degrees
- moved C7 64.8 mm to (145.0, 94.0), turned to 90 degrees
- moved C8 63.2 mm to (146.2, 94.0), turned to 90 degrees
- moved C3 63.0 mm to (143.6, 95.8), turned to 180 degrees
- moved C9 61.8 mm to (147.4, 94.0), turned to 90 degrees
- moved C12 58.9 mm to (151.4, 106.0), turned to -90 degrees
- moved C10 58.0 mm to (151.0, 94.0), turned to 90 degrees
- moved C11 52.4 mm to (157.0, 99.0)
- moved C4 49.8 mm to (157.0, 97.8)
- moved R7 29.8 mm to (157.0, 100.2)
- moved C17 28.2 mm to (159.4, 100.2)
- moved Y1 22.8 mm to (158.2, 102.6)
- moved C16 21.4 mm to (158.2, 105.0)
- moved SW3 9.17 mm to (112.2, 128.0)
- moved U1 2.50 mm to (141.2, 108.6)
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Routing:
- net +3V3: track 0.00 -> 20.3 mm, vias 0 -> 6
- net GND: track 0.00 -> 10.1 mm, vias 0 -> 17
- net +1V1: track 0.00 -> 6.81 mm, vias 0 -> 2
- net Net-(U3-XIN): track 0.00 -> 5.85 mm
- net QSPI_SD3: track 0.00 -> 5.56 mm
- net QSPI_SCLK: track 0.00 -> 4.90 mm
- net QSPI_SD0: track 0.00 -> 4.24 mm
- net unconnected-(U3-GPIO12-Pad15): track 0.00 -> 3.98 mm
- net QSPI_SD2: track 0.00 -> 3.57 mm
- net unconnected-(U3-GPIO14-Pad17): track 0.00 -> 3.37 mm
- net unconnected-(U3-GPIO9-Pad12): track 0.00 -> 3.13 mm
- net Net-(C17-Pad1): track 0.00 -> 3.12 mm
- net Net-(U3-USB_DM): track 0.00 -> 3.12 mm
- net Net-(U3-XOUT): track 0.00 -> 3.05 mm
- net unconnected-(U3-GPIO11-Pad14): track 0.00 -> 2.96 mm
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- added copper zone on In1.Cu, net GND
Other:
- board outline added: 150 x 90 mm

Commit message: board wip
Parts:
- J2: footprint Connector_PinHeader_2.54mm:PinHeader_1x26_P2.54mm_Vertical -> Connector_PinHeader_2.54mm:PinHeader_1x22_P2.54mm_Vertical
- J5: value Conn_ARM_JTAG_SWD_10 -> SWD
- moved J5 23.7 mm to (158.8, 90.0)
- moved C2 8.30 mm to (139.0, 111.6)
- moved C1 5.35 mm to (136.8, 111.6), turned to 180 degrees
- moved U1 1.00 mm to (140.4, 108.0), turned to 180 degrees
- moved C11 0.72 mm to (156.4, 99.4)
- moved C16 0.72 mm to (157.6, 105.4)
- moved C4 0.72 mm to (156.4, 98.2)
- moved Y1 0.72 mm to (157.6, 103.0)
- moved C17 0.72 mm to (158.8, 100.6)
- moved R7 0.72 mm to (156.4, 100.6)
Connections:
- J2 pad 1: unconnected-(J2-Pin_1-Pad1) -> +5V
- J2 pad 10: unconnected-(J2-Pin_10-Pad10) -> GPIO05
- J2 pad 11: unconnected-(J2-Pin_11-Pad11) -> GPIO06
- J2 pad 12: unconnected-(J2-Pin_12-Pad12) -> GPIO07
- J2 pad 13: unconnected-(J2-Pin_13-Pad13) -> GND
- J2 pad 14: unconnected-(J2-Pin_14-Pad14) -> GPIO08
- J2 pad 15: unconnected-(J2-Pin_15-Pad15) -> GPIO09
- J2 pad 16: unconnected-(J2-Pin_16-Pad16) -> GPIO10
- J2 pad 17: unconnected-(J2-Pin_17-Pad17) -> GPIO11
- J2 pad 18: unconnected-(J2-Pin_18-Pad18) -> GPIO12
- J2 pad 19: unconnected-(J2-Pin_19-Pad19) -> GPIO13
- J2 pad 2: unconnected-(J2-Pin_2-Pad2) -> +3V3
- J2 pad 20: unconnected-(J2-Pin_20-Pad20) -> GPIO14
- J2 pad 21: unconnected-(J2-Pin_21-Pad21) -> GPIO15
- J2 pad 22: unconnected-(J2-Pin_22-Pad22) -> GND
- J2 pad 3: unconnected-(J2-Pin_3-Pad3) -> GND
- J2 pad 4: unconnected-(J2-Pin_4-Pad4) -> GND
- J2 pad 5: unconnected-(J2-Pin_5-Pad5) -> GPIO00
- J2 pad 6: unconnected-(J2-Pin_6-Pad6) -> GPIO01
- J2 pad 7: unconnected-(J2-Pin_7-Pad7) -> GPIO02
- J2 pad 8: unconnected-(J2-Pin_8-Pad8) -> GPIO03
- J2 pad 9: unconnected-(J2-Pin_9-Pad9) -> GPIO04
- U3 pad 11: unconnected-(U3-GPIO8-Pad11) -> GPIO08
- U3 pad 12: unconnected-(U3-GPIO9-Pad12) -> GPIO09
- U3 pad 13: unconnected-(U3-GPIO10-Pad13) -> GPIO10
- U3 pad 14: unconnected-(U3-GPIO11-Pad14) -> GPIO11
- U3 pad 15: unconnected-(U3-GPIO12-Pad15) -> GPIO12
- U3 pad 16: unconnected-(U3-GPIO13-Pad16) -> GPIO13
- U3 pad 17: unconnected-(U3-GPIO14-Pad17) -> GPIO14
- U3 pad 18: unconnected-(U3-GPIO15-Pad18) -> GPIO15
- U3 pad 2: unconnected-(U3-GPIO0-Pad2) -> GPIO00
- U3 pad 3: unconnected-(U3-GPIO1-Pad3) -> GPIO01
- U3 pad 4: unconnected-(U3-GPIO2-Pad4) -> GPIO02
- U3 pad 5: unconnected-(U3-GPIO3-Pad5) -> GPIO03
- U3 pad 6: unconnected-(U3-GPIO4-Pad6) -> GPIO04
- U3 pad 7: unconnected-(U3-GPIO5-Pad7) -> GPIO05
- U3 pad 8: unconnected-(U3-GPIO6-Pad8) -> GPIO06
- U3 pad 9: unconnected-(U3-GPIO7-Pad9) -> GPIO07
Routing:
- net QSPI_SD3: track 5.56 -> 17.4 mm
- net GND: track 10.1 -> 21.0 mm, vias 17 -> 30
- net QSPI_SCLK: track 4.90 -> 15.0 mm
- net QSPI_SD0: track 4.24 -> 12.2 mm
- net QSPI_SS: track 2.03 -> 8.47 mm
- net QSPI_SD1: track 2.91 -> 8.28 mm
- net unconnected-(U3-GPIO12-Pad15): track 3.98 -> 0.00 mm
- net GPIO12: track 0.00 -> 3.98 mm
- net QSPI_SD2: track 3.57 -> 7.53 mm
- net unconnected-(U3-GPIO14-Pad17): track 3.37 -> 0.00 mm
- net GPIO14: track 0.00 -> 3.37 mm
- net SWCLK: track 0.00 -> 3.14 mm
- net unconnected-(U3-GPIO9-Pad12): track 3.13 -> 0.00 mm
- net GPIO09: track 0.00 -> 3.13 mm
- net +1V1: track 6.81 -> 9.79 mm, vias 2 -> 3
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
Commit message: board wip
Parts:
- moved C14 73.4 mm to (149.2, 70.7)
- moved C15 73.4 mm to (149.2, 72.7)
- moved D1 73.4 mm to (161.8, 72.7)
- moved D2 73.4 mm to (161.8, 77.2)
- moved R3 73.4 mm to (148.8, 75.2)
- moved R6 73.4 mm to (148.8, 77.7)
- moved U2 73.4 mm to (140.7, 72.0)
- moved R13 21.9 mm to (129.7, 76.0)
- moved R12 21.9 mm to (128.9, 78.9)
- moved J2 21.0 mm to (124.9, 117.4)
- moved J1 20.0 mm to (112.5, 83.2), turned to 180 degrees
- moved D5 19.6 mm to (128.0, 110.6)
- moved R2 19.2 mm to (142.2, 104.4)
- moved R1 16.3 mm to (140.0, 104.4)
- moved SW1 13.8 mm to (104.8, 116.0)
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Routing:
- net GPIO00: track 2.56 -> 20.4 mm
- net GPIO01: track 2.56 -> 17.8 mm
- net GPIO02: track 2.56 -> 15.9 mm
- net GPIO03: track 2.56 -> 13.9 mm
- net GPIO04: track 2.56 -> 12.6 mm
- net QSPI_SS: track 8.47 -> 16.6 mm
- net #USB_BOOT: track 0.00 -> 0.69 mm, vias 0 -> 1
Other:
- board size 150 x 90 mm -> 150 x 71 mm
- board text added: "5V 3V3 GND GND GP00 GP01 GP02 GP03 GP04 GP05 GP06 GP07"

Commit message: board wip
Parts:
- removed the J1 at (213.1, 95.9)
- moved J4 68.5 mm to (134.0, 76.0), turned to 90 degrees
- moved D2 36.9 mm to (127.0, 89.4), turned to 180 degrees
- moved D1 35.1 mm to (127.2, 78.6), turned to 180 degrees
- moved J3 29.2 mm to (169.2, 76.0), turned to -90 degrees
- moved R3 22.4 mm to (128.8, 85.2)
- moved C15 22.1 mm to (133.4, 88.2)
- moved C14 20.9 mm to (137.8, 88.2)
- moved R6 20.5 mm to (128.8, 82.2)
- moved R8 20.1 mm to (152.8, 98.2)
- moved SW2 17.4 mm to (158.8, 103.5)
- moved R12 15.0 mm to (124.4, 93.2), turned to -90 degrees
- moved U2 12.6 mm to (135.0, 83.2), turned to 180 degrees
- moved R9 11.9 mm to (165.2, 93.2), turned to 90 degrees
- moved R10 9.12 mm to (167.2, 93.2), turned to 90 degrees
- moved R13 8.67 mm to (125.6, 83.7), turned to 90 degrees
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Connections:
- U3 pad 28: OLED_SCK -> LED_D1
- U3 pad 29: OLED_SDA -> LED_D2
- U3 pad 36: LED_D2 -> OLED_SDA
- U3 pad 37: LED_D1 -> OLED_SCK
Routing:
- net ELRS_TX: track 0.00 -> 33.0 mm
- net ELRS_RX: track 0.00 -> 30.7 mm
- net GPIO15: track 1.12 -> 29.9 mm, vias 1 -> 2
- net LED_D2: track 0.00 -> 26.3 mm
- net LED_D1: track 0.00 -> 24.7 mm
- net OLED_SCK: track 0.00 -> 24.5 mm
- net OLED_SDA: track 0.00 -> 23.6 mm
- net GPIO14: track 3.37 -> 26.5 mm
- net GPIO13: track 2.91 -> 23.6 mm
- net RUN: track 1.04 -> 21.1 mm, vias 1 -> 2
- net GPIO10: track 1.04 -> 19.4 mm, vias 1 -> 2
- net GPIO08: track 1.04 -> 18.0 mm, vias 1 -> 2
- net GPIO12: track 3.98 -> 20.1 mm
- net GPIO11: track 2.96 -> 18.4 mm
- net GPIO09: track 3.13 -> 17.3 mm
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Other:
- board size 150 x 71 mm -> 75 x 48 mm
- board text added: "5V 3V3 GND GND GP00 GP01 GP02 GP03 GP04 GP05 GP06 GP07 GND GP08 GP09 GP10 GP11 GP12 GP13 GP14 GP15 GND"
- board text removed: "5V 3V3 GND GND GP00 GP01 GP02 GP03 GP04 GP05 GP06 GP07"

Commit message: board wip
Parts:
- R11: footprint Resistor_SMD:R_0402_1005Metric -> Resistor_SMD:R_0603_1608Metric
- moved C18 7.86 mm to (119.2, 107.2), turned to -90 degrees
- moved C14 5.37 mm to (133.0, 90.6)
- moved C19 5.24 mm to (119.2, 103.8), turned to 90 degrees
- moved R11 4.44 mm to (116.0, 107.2), turned to -90 degrees
- moved U4 3.62 mm to (125.0, 105.4)
- moved D5 2.98 mm to (123.8, 111.2)
- moved U2 2.40 mm to (135.0, 85.6)
- moved R12 2.34 mm to (125.2, 95.4), turned to 90 degrees
- moved D1 2.00 mm to (127.2, 80.6)
- moved R13 2.00 mm to (125.6, 85.7)
- moved R3 2.00 mm to (128.8, 87.2)
- moved R6 2.00 mm to (128.8, 84.2)
- moved D2 1.22 mm to (127.2, 90.6)
- moved C15 1.08 mm to (133.0, 89.2)
Connections:
- net USB_DM renamed USB_D-
- net USB_DP renamed USB_D+
- J2 pad 1: +5V -> VBUS
- J2 pad 2: +3V3 -> +5V
- J2 pad 3: GND -> +3V3
- U3 pad 38: unconnected-(U3-GPIO26_ADC0-Pad38) -> RS485_TXD
- U3 pad 39: unconnected-(U3-GPIO27_ADC1-Pad39) -> RS485_RE_NDE
- U3 pad 40: unconnected-(U3-GPIO28_ADC2-Pad40) -> RS485_RXD
Routing:
- net +5V: track 0.00 -> 93.7 mm, vias 0 -> 2
- net GND: track 23.0 -> 80.5 mm, vias 32 -> 49
- net USB_D-: track 0.00 -> 38.6 mm
- net USB_D+: track 0.00 -> 38.4 mm
- net +3V3: track 21.8 -> 56.8 mm, vias 7 -> 11
- net VBUS: track 0.00 -> 30.2 mm, vias 0 -> 2
- net Net-(J1-Pad2): track 0.00 -> 17.0 mm
- net Net-(J1-Pad1): track 0.00 -> 13.3 mm
- net Net-(J1-Pad3): track 0.00 -> 9.41 mm
- net Net-(D1-K): track 0.00 -> 6.99 mm
- net Net-(D2-K): track 0.00 -> 6.88 mm
- net Net-(SW3-B): track 0.69 -> 6.69 mm
- net #USB_BOOT: track 0.69 -> 6.69 mm
Other:
- board text added: "VBUS 5V 3V3 GND GP00 GP01 GP02 GP03 GP04 GP05 GP06 GP07 GND GP08 GP09 GP10 GP11 GP12 GP13 GP14 GP15 GND"
- board text removed: "5V 3V3 GND GND GP00 GP01 GP02 GP03 GP04 GP05 GP06 GP07 GND GP08 GP09 GP10 GP11 GP12 GP13 GP14 GP15 GND"

Commit message: board rc1
Routing:
- net +3V3: track 56.8 -> 169.6 mm, vias 11 -> 13
- net Net-(SW3-B): track 6.69 -> 60.8 mm, vias 1 -> 2
- net #USB_BOOT: track 6.69 -> 45.0 mm, vias 1 -> 2
- net RE_SW: track 1.20 -> 32.3 mm
- net RS485_RE_NDE: track 0.00 -> 24.0 mm
- net RE_B: track 1.20 -> 24.8 mm
- net RS485_TXD: track 0.00 -> 19.4 mm
- net +1V1: track 9.79 -> 26.9 mm
- net RS485_RXD: track 0.00 -> 16.8 mm
- net RE_A: track 1.20 -> 16.3 mm
- net GPIO12: track 20.1 -> 25.0 mm
- net GPIO13: track 23.6 -> 28.2 mm
- net GPIO14: track 26.5 -> 30.9 mm
- net GPIO15: track 29.9 -> 33.8 mm
- net GPIO11: track 18.4 -> 21.9 mm
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- added copper zone on F.Cu, net GND
- added copper zone on In2.Cu, net GND

Commit message: board rc2
Routing:
- net #USB_BOOT: track 45.0 -> 48.0 mm
- net GND: vias 66 -> 69
Changed lines of the file:
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@@
     (effects (font (size 0.79 0.79) (thickness 0.15)) (justify left bottom))
   )
-  (segment (start 124.08 116.92) (end 124.08 118.325) (width 0.4) (layer "F.Cu") (net 1))
   (segment (start 147.4 104.5625) (end 147.4 105.325) (width 0.2) (layer "F.Cu") (net 1))
   (segment (start 151.4 100.925) (end 151.6 100.725) (width 0.2) (layer "F.Cu") (net 1))
@@
   (segment (start 120.175 104.575) (end 120.975 105.375) (width 0.4) (layer "F.Cu") (net 1))
   (segment (start 147.4 105.325) (end 147.8 105.725) (width 0.2) (layer "F.Cu") (net 1))
-  (segment (start 130 111) (end 124.08 116.92) (width 0.4) (layer "F.Cu") (net 1))
+  (segment (start 124.08 118.325) (end 124.08 116.92) (width 0.6) (layer "F.Cu") (net 1))
   (segment (start 142.4 98.525) (end 142 98.125) (width 0.2) (layer "F.Cu") (net 1))
   (segment (start 142.6 95.605) (end 142.6 95.925) (width 0.2) (layer "F.Cu") (net 1))
@@
   (segment (start 123.175 105.375) (end 124 106.2) (width 0.6) (layer "F.Cu") (net 1))
   (segment (start 135.8 107.2) (end 135.8 105.615) (width 0.2) (layer "F.Cu") (net 1))
+  (segment (start 124.08 116.92) (end 130 111) (width 0.6) (layer "F.Cu") (net 1))
   (segment (start 119.2 104.575) (end 120.175 104.575) (width 0.4) (layer "F.Cu") (net 1))
   (segment (start 143.8 96.525) (end 143.8 95.605) (width 0.2) (layer "F.Cu") (net 1))
@@
   (via (at 115 111) (size 0.6) (drill 0.3) (layers "F.Cu" "B.Cu") (free) (net 2))
   (via (at 143.8 93.925) (size 0.4) (drill 0.2) (layers "F.Cu" "B.Cu") (free) (net 2))
+  (via (at 106 81) (size 0.6) (drill 0.3) (layers "F.Cu" "B.Cu") (free) (net 2))
   (via (at 156.4 101.725) (size 0.4) (drill 0.2) (layers "F.Cu" "B.Cu") (free) (net 2))
+  (via (at 106 95) (size 0.6) (drill 0.3) (layers "F.Cu" "B.Cu") (free) (net 2))
   (via (at 125.2 93) (size 0.6) (drill 0.3) (layers "F.Cu" "B.Cu") (net 2))
   (via (at 132 95) (size 0.6) (drill 0.3) (layers "F.Cu" "B.Cu") (free) (net 2))
@@
   (via (at 147 100.525) (size 0.4) (drill 0.2) (layers "F.Cu" "B.Cu") (net 2))
   (via (at 114.8 113.4) (size 0.6) (drill 0.3) (layers "F.Cu" "B.Cu") (free) (net 2))
+  (via (at 106 75) (size 0.6) (drill 0.3) (layers "F.Cu" "B.Cu") (free) (net 2))
   (via (at 157 103.2) (size 0.4) (drill 0.2) (layers "F.Cu" "B.Cu") (free) (net 2))
   (via (at 157 108) (size 0.4) (drill 0.2) (layers "F.Cu" "B.Cu") (free) (net 2))
@@
   (segment (start 147.989339 102.475) (end 150.539339 99.925) (width 0.6) (layer "In2.Cu") (net 3))
   (segment (start 127.8 96.2) (end 127.2 96.2) (width 0.4) (layer "F.Cu") (net 4))
-  (segment (start 121.8 111.175) (end 121.8 118.065) (width 0.4) (layer "F.Cu") (net 4))
+  (segment (start 121.85 107.675) (end 124.725 107.675) (width 0.6) (layer "F.Cu") (net 4))
   (segment (start 135 81.2) (end 135 86.6) (width 0.4) (layer "F.Cu") (net 4))
-  (segment (start 127.2 101) (end 125.8 102.4) (width 0.4) (layer "F.Cu") (net 4))
-  (segment (start 125.8 102.4) (end 125.8 106) (width 0.4) (layer "F.Cu") (net 4))
-  (segment (start 121.85 111.125) (end 121.8 111.175) (width 0.4) (layer "F.Cu") (net 4))
+  (segment (start 121.8 118.065) (end 121.54 118.325) (width 0.6) (layer "F.Cu") (net 4))
+  (segment (start 121.85 107.675) (end 121.85 111.125) (width 0.6) (layer "F.Cu") (net 4))
+  (segment (start 121.85 111.125) (end 121.8 111.175) (width 0.6) (layer "F.Cu") (net 4))
+  (segment (start 126 106.4) (end 126 102.2) (width 0.6) (layer "F.Cu") (net 4))
   (segment (start 131.4 74.6) (end 131.4 77.6) (width 0.4) (layer "F.Cu") (net 4))
   (segment (start 121.075 107.675) (end 121.85 107.675) (width 0.4) (layer "F.Cu") (net 4))
   (segment (start 131.4 77.6) (end 135 81.2) (width 0.4) (layer "F.Cu") (net 4))
+  (segment (start 124.725 107.675) (end 126 106.4) (width 0.6) (layer "F.Cu") (net 4))
+  (segment (start 121.8 111.175) (end 121.8 118.065) (width 0.6) (layer "F.Cu") (net 4))
   (segment (start 132.52 91.48) (end 127.8 96.2) (width 0.4) (layer "F.Cu") (net 4))
   (segment (start 134.095 87.505) (end 132.525 87.505) (width 0.4) (layer "F.Cu") (net 4))
@@
   (segment (start 132.6 73.4) (end 131.4 74.6) (width 0.4) (layer "F.Cu") (net 4))
   (segment (start 132.52 89.2) (end 132.52 87.51) (width 0.4) (layer "F.Cu") (net 4))
-  (segment (start 124.125 107.675) (end 121.85 107.675) (width 0.4) (layer "F.Cu") (net 4))
   (segment (start 119.425 106.425) (end 120.675 107.675) (width 0.6) (layer "F.Cu") (net 4))
-  (segment (start 125.8 106) (end 124.125 107.675) (width 0.4) (layer "F.Cu") (net 4))
   (segment (start 132.52 89.2) (end 132.52 90.6) (width 0.4) (layer "F.Cu") (net 4))
   (segment (start 120.675 107.675) (end 121.85 107.675) (width 0.6) (layer "F.Cu") (net 4))
   (segment (start 164.12 76) (end 161.52 73.4) (width 0.4) (layer "F.Cu") (net 4))
-  (segment (start 121.85 107.675) (end 121.85 111.125) (width 0.4) (layer "F.Cu") (net 4))
+  (segment (start 126 102.2) (end 127.2 101) (width 0.6) (layer "F.Cu") (net 4))
   (segment (start 119.15 106.375) (end 119.2 106.425) (width 0.6) (layer "F.Cu") (net 4))
   (segment (start 132.52 90.6) (end 132.52 91.48) (width 0.4) (layer "F.Cu") (net 4))
-  (segment (start 121.8 118.065) (end 121.54 118.325) (width 0.4) (layer "F.Cu") (net 4))
   (segment (start 135 86.6) (end 134.095 87.505) (width 0.4) (layer "F.Cu") (net 4))
   (segment (start 132.52 87.51) (end 132.525 87.505) (width 0.4) (layer "F.Cu") (net 4))
@@
   (segment (start 150.475 99.325) (end 152.4 97.4) (width 0.2) (layer "B.Cu") (net 22))
   (segment (start 148.8 99.325) (end 150.475 99.325) (width 0.2) (layer "B.Cu") (net 22))
-  (segment (start 116 108.8) (end 119 111.8) (width 0.4) (layer "F.Cu") (net 23))
+  (segment (start 119 118.325) (end 119 111.8) (width 0.6) (layer "F.Cu") (net 23))
   (segment (start 116 108.025) (end 116 108.8) (width 0.4) (layer "F.Cu") (net 23))
   (segment (start 106.725 103.2) (end 110 103.2) (width 0.4) (layer "F.Cu") (net 23))
   (segment (start 115.975 108) (end 116 108.025) (width 0.6) (layer "F.Cu") (net 23))
-  (segment (start 119 111.8) (end 119 118.325) (width 0.4) (layer "F.Cu") (net 23))
   (segment (start 106.725 108) (end 113.2 108) (width 0.4) (layer "F.Cu") (net 23))
   (segment (start 113.2 108) (end 115.975 108) (width 0.6) (layer "F.Cu") (net 23))
+  (segment (start 119 111.8) (end 116 108.8) (width 0.6) (layer "F.Cu") (net 23))
   (via (at 110 103.2) (size 0.6) (drill 0.3) (layers "F.Cu" "B.Cu") (net 23))
   (via (at 113.2 108) (size 0.6) (drill 0.3) (layers "F.Cu" "B.Cu") (net 23))
@@
   (via (at 139.8 105.525) (size 0.4) (drill 0.2) (layers "F.Cu" "B.Cu") (free) (net 29))
   (via (at 116.6 115.8) (size 0.4) (drill 0.2) (layers "F.Cu" "B.Cu") (net 29))
-  (segment (start 120.225 112.175) (end 133.15 112.175) (width 0.2) (layer "B.Cu") (net 29))
-  (segment (start 116.6 115.8) (end 120.225 112.175) (width 0.2) (layer "B.Cu") (net 29))
-  (segment (start 133.15 112.175) (end 139.8 105.525) (width 0.2) (layer "B.Cu") (net 29))
+  (segment (start 139.8 110.6) (end 139.8 105.525) (width 0.2) (layer "B.Cu") (net 29))
+  (segment (start 136 114.4) (end 139.8 110.6) (width 0.2) (layer "B.Cu") (net 29))
+  (segment (start 116.6 115.8) (end 118 114.4) (width 0.2) (layer "B.Cu") (net 29))
+  (segment (start 118 114.4) (end 136 114.4) (width 0.2) (layer "B.Cu") (net 29))
   (segment (start 142.9625 100.125) (end 141.577818 100.125) (width 0.2) (layer "F.Cu") (net 30))
   (segment (start 140.777818 99.325) (end 140.51 99.325) (width 0.2) (layer "F.Cu") (net 30))
@@
   (segment (start 146.377818 115.4) (end 118.2 115.4) (width 0.2) (layer "B.Cu") (net 33))
   (segment (start 153.4 98.8) (end 153.4 108.377818) (width 0.2) (layer "B.Cu") (net 33))
+  (segment (start 149.8375 98.525) (end 149.4 98.0875) (width 0.2) (layer "F.Cu") (net 34))
+  (segment (start 162.2 88.6) (end 165.2 91.6) (width 0.2) (layer "F.Cu") (net 34))
+  (segment (start 165.2 91.6) (end 165.2 92.69) (width 0.2) (layer "F.Cu") (net 34))
   (segment (start 154.74 88.6) (end 162.2 88.6) (width 0.2) (layer "F.Cu") (net 34))
-  (segment (start 149.8375 93.5025) (end 154.74 88.6) (width 0.2) (layer "F.Cu") (net 34))
-  (segment (start 165.2 91.6) (end 165.2 92.69) (width 0.2) (layer "F.Cu") (net 34))
-  (segment (start 149.8375 98.525) (end 149.8375 93.5025) (width 0.2) (layer "F.Cu") (net 34))
-  (segment (start 162.2 88.6) (end 165.2 91.6) (width 0.2) (layer "F.Cu") (net 34))
+  (segment (start 149.4 98.0875) (end 149.4 93.94) (width 0.2) (layer "F.Cu") (net 34))
+  (segment (start 149.4 93.94) (end 154.74 88.6) (width 0.2) (layer "F.Cu") (net 34))
   (segment (start 149 97.6875) (end 149 93.774315) (width 0.2) (layer "F.Cu") (net 35))
   (segment (start 162.71 88.2) (end 167.2 92.69) (width 0.2) (layer "F.Cu") (net 35))
