File: pcb/rp2040-board.kicad_pcb (KiCad board)
At the start: 4 copper layers, 65 x 56 mm, 52 parts, among them J1 Conn_01x10, J3 OLED, J4 Conn_01x08, J5 PWR IN, J6 Raspberry_Pi_4, Q1 AO3401A, SW1 TS-1187A-B-A-B, U1 DRV8837, U2 DRV8837, U3 DRV8837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

Commit message: board final touches
Parts:
- C11: value 22uF -> 10uF
- moved R3 0.50 mm to (164.0, 98.0)
- moved TP1 0.50 mm to (124.5, 80.5)
Routing:
- net +5V: track 15.3 -> 19.3 mm, vias 11 -> 13
- net RUN: track 10.4 -> 10.9 mm
- net Net-(SW1-B): track 8.04 -> 7.54 mm
Other:
- board text added: "GND 12-24V"
- board text added: "github.com/barycz/rp2040-board Tomas Barak, 2025"
- board text removed: "github.com/barycz/rp2040-board Tomas Barak, 2024"
Changed lines of the file:
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@@
 			)
 		)
+		(property "LCSC Part" "C15127"
+			(at 0 0 180)
+			(unlocked yes)
+			(layer "F.Fab")
+			(hide yes)
+			(effects
+				(font
+					(size 1 1)
+					(thickness 0.15)
+				)
+			)
+		)
 		(property ki_fp_filters "SOT?23*")
 		(sheetname "/Power/")
@@
 	(footprint "TestPoint:TestPoint_Pad_D1.0mm"
 		(layer "F.Cu")
-		(at 124 80.5)
+		(at 124.5 80.5)
 		(descr "SMD pad as test Point, diameter 1.0mm")
 		(tags "test point SMD pad")
@@
 		(sheetname "/Power/")
 		(sheetfile "power.kicad_sch")
-		(attr exclude_from_pos_files)
+		(attr exclude_from_pos_files exclude_from_bom)
 		(fp_circle
 			(center 0 0)
@@
 		(sheetname "/Motor Drivers/")
 		(sheetfile "motor_drivers.kicad_sch")
-		(attr through_hole)
+		(attr through_hole exclude_from_bom)
 		(fp_line
 			(start -1.38 -1.38)
@@
 		(sheetname "/")
 		(sheetfile "rp2040-board.kicad_sch")
-		(attr exclude_from_pos_files)
+		(attr exclude_from_pos_files exclude_from_bom)
 		(fp_circle
 			(center 0 0)
@@
 		(sheetname "/Power/")
 		(sheetfile "power.kicad_sch")
-		(attr through_hole)
+		(attr through_hole exclude_from_bom)
 		(fp_line
 			(start 7.71 -2.71)
@@
 			)
 		)
-		(property "Value" "22uF"
+		(property "Value" "10uF"
 			(at 0 1.68 90)
 			(layer "F.Fab")
@@
 			)
 		)
-		(property "LCSC Part" "C45783"
+		(property "LCSC Part" "C440198"
 			(at 0 0 90)
 			(unlocked yes)
@@
 		(sheetname "/")
 		(sheetfile "rp2040-board.kicad_sch")
-		(attr through_hole)
+		(attr through_hole exclude_from_bom)
 		(fp_line
 			(start -1.33 8.95)
@@
 		(sheetname "/")
 		(sheetfile "rp2040-board.kicad_sch")
-		(attr smd)
+		(attr smd exclude_from_bom)
 		(fp_line
 			(start -10.61 -23.07)
@@
 		(tags "test point SMD pad")
 		(property "Reference" "TP4"
-			(at -1.5 1.5 0)
+			(at -0.5 -2.5 90)
 			(layer "F.SilkS")
 			(effects
@@
 		(sheetname "/")
 		(sheetfile "rp2040-board.kicad_sch")
-		(attr exclude_from_pos_files)
+		(attr exclude_from_pos_files exclude_from_bom)
 		(fp_circle
 			(center 0 0)
@@
 	(footprint "Resistor_SMD:R_0402_1005Metric"
 		(layer "F.Cu")
-		(at 164 97.5 -90)
+		(at 164 98 -90)
 		(descr "Resistor SMD 0402 (1005 Metric), square (rectangular) end terminal, IPC-7351 nominal, (Body size source: IPC-SM-782 page 72, https://www.pcb-3d.com/wordpress/wp-content/uploads/ipc-sm-782a_amendment_1_and_2.pdf), generated with kicad-footprint-generator")
 		(tags "resistor")
 		(property "Reference" "R3"
-			(at 1 2 180)
+			(at 0.5 2 180)
 			(layer "F.SilkS")
 			(effects
@@
 		(tags "test point SMD pad")
 		(property "Reference" "TP3"
-			(at -2.5 0 0)
+			(at -0.5 -2 0)
 			(layer "F.SilkS")
 			(effects
@@
 		(sheetname "/")
 		(sheetfile "rp2040-board.kicad_sch")
-		(attr exclude_from_pos_files)
+		(attr exclude_from_pos_files exclude_from_bom)
 		(fp_circle
 			(center 0 0)
@@
 		)
 		(fp_text user "${REFERENCE}"
-			(at -2.5 0 0)
-			(layer "F.Fab")
+			(at 0 -2.5 0)
+			(layer "User.1")
 			(effects
 				(font
@@
 		(sheetname "/")
 		(sheetfile "rp2040-board.kicad_sch")
-		(attr through_hole)
+		(attr through_hole exclude_from_bom)
 		(fp_line
 			(start -1.38 -1.38)
@@
 		(sheetname "/Power/")
 		(sheetfile "power.kicad_sch")
-		(attr through_hole)
+		(attr through_hole exclude_from_bom)
 		(fp_line
 			(start -3.87 1.33)
@@
 		)
 	)
+	(gr_text "GND   12-24V"
+		(at 108 110 90)
+		(layer "F.SilkS")
+		(effects
+			(font
+				(size 0.79 0.79)
+				(thickness 0.15)
+			)
+			(justify left bottom)
+		)
+	)
 	(gr_text "1A\n\n1B\n\n2A\n\n2B\n\n3A\n\n3B\n\n4A\n\n4B"
 		(at 130 119.75 90)
@@
 		)
 	)
-	(gr_text "github.com/barycz/rp2040-board\nTomas Barak, 2024"
-		(at 160.5 111.5 0)
+	(gr_text "github.com/barycz/rp2040-board\nTomas Barak, 2025"
+		(at 163.5 112.5 0)
 		(layer "B.SilkS")
 		(effects
@@
 	)
 	(segment
+		(start 110 114)
+		(end 109 114)
+		(width 0.6)
+		(layer "F.Cu")
+		(net 4)
+	)
+	(segment
 		(start 116 113.5)
 		(end 115.5 114)
@@
 	)
 	(segment
+		(start 115.5 114)
+		(end 114.5 114)
+		(width 0.6)
+		(layer "F.Cu")
+		(net 4)
+	)
+	(segment
 		(start 127.02 113.48)
 		(end 126.5 114)
@@
 	)
 	(segment
+		(start 126.5 114)
+		(end 125.5 114)
+		(width 0.6)
+		(layer "F.Cu")
+		(net 4)
+	)
+	(segment
 		(start 111.7 113.5)
 		(end 111 113.5)
@@
 		(net 4)
 	)
+	(segment
+		(start 121 114)
+		(end 120 114)
+		(width 0.6)
+		(layer "F.Cu")
+		(net 4)
+	)
 	(via
 		(at 121 82)
@@
 	)
 	(via
-		(at 122.5 80)
+		(at 123 80)
 		(size 0.6)
 		(drill 0.3)
@@
 	)
 	(via
+		(at 114.5 114)
+		(size 0.6)
+		(drill 0.3)
+		(layers "F.Cu" "B.Cu")
+		(net 4)
+	)
+	(via
 		(at 115.5 114)
 		(size 0.6)
@@
 	)
 	(via
-		(at 122.5 82)
+		(at 123 82)
 		(size 0.6)
 		(drill 0.3)
@@
 	)
 	(via
-		(at 121 84)
+		(at 122 81)
 		(size 0.6)
 		(drill 0.3)
@@
 	)
 	(via
-		(at 124 82)
+		(at 120 114)
 		(size 0.6)
 		(drill 0.3)
 		(layers "F.Cu" "B.Cu")
-		(free yes)
 		(net 4)
 	)
 	(via
-		(at 122.5 84)
+		(at 109 114)
+		(size 0.6)
+		(drill 0.3)
+		(layers "F.Cu" "B.Cu")
+		(net 4)
+	)
+	(via
+		(at 125.5 114)
 		(size 0.6)
 		(drill 0.3)
 		(layers "F.Cu" "B.Cu")
-		(free yes)
 		(net 4)
 	)
@@
 	)
 	(segment
-		(start 164 96.99)
-		(end 164 96.660818)
+		(start 160.311786 94.679)
+		(end 156.902786 91.27)
 		(width 0.4)
 		(layer "F.Cu")
@@
 	)
 	(segment
-		(start 160.311786 94.679)
-		(end 156.902786 91.27)
+		(start 164 96.660818)
+		(end 164 97.49)
 		(width 0.4)
 		(layer "F.Cu")
@@
 	)
 	(segment
-		(start 163.875 100)
-		(end 163.875 98.135)
+		(start 164 99.875)
+		(end 163.875 100)
 		(width 0.4)
 		(layer "F.Cu")
@@
 	)
 	(segment
-		(start 163.875 106)
-		(end 163.875 100)
+		(start 164 98.51)
+		(end 164 99.875)
 		(width 0.4)
 		(layer "F.Cu")
@@
 	)
 	(segment
-		(start 163.875 98.135)
-		(end 164 98.01)
+		(start 163.875 106)
+		(end 163.875 100)
 		(width 0.4)
 		(layer "F.Cu")
@@
 		(polygon
 			(pts
-				(xy 100 64) (xy 165 64) (xy 165 107) (xy 137 107) (xy 137 120) (xy 100 120)
+				(xy 100 64) (xy 165 64) (xy 165 104.5) (xy 163 106.5) (xy 138.5 106.5) (xy 136.5 108.5) (xy 136.5 118)
+				(xy 134.5 120) (xy 100 120)
 			)
 		)
@@
 		(polygon
 			(pts
-				(xy 100 64) (xy 165 64) (xy 165 107) (xy 137 107) (xy 137 120) (xy 100 120)
+				(xy 100 64) (xy 165 64) (xy 165 104.5) (xy 163 106.5) (xy 138.5 106.5) (xy 136.5 108.5) (xy 136.5 118)
+				(xy 134.5 120) (xy 100 120)
 			)
 		)

Commit message: board rc1
Parts:
- added G***: LOGO, gfx:robot1, B.Cu at (134.3, 89.8)

Commit message: board rc2
Parts:
- R5: value 1k -> 3k3
- R6: value 2k2 -> 100k
- moved R6 2.24 mm to (117.5, 79.0)
Connections:
- R5 pad 2: Net-(R5-Pad2) -> GND
- R6 pad 1: Net-(R5-Pad2) -> Net-(U5-VSENSE)
Routing:
- net GND: track 60.3 -> 63.4 mm
- net Net-(U5-VSENSE): track 11.2 -> 12.8 mm
- net Net-(R5-Pad2): track 0.98 -> 0.00 mm
Changed lines of the file:
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@@
 	(net 52 "Net-(U5-VSENSE)")
 	(net 53 "DRVNSLEEP")
-	(net 54 "Net-(R5-Pad2)")
-	(net 55 "unconnected-(U5-NC-Pad3)")
-	(net 56 "unconnected-(U5-EN-Pad5)")
-	(net 57 "LED_DIN")
-	(net 58 "unconnected-(U5-NC-Pad2)")
-	(net 59 "LED_DOUT")
-	(net 60 "PICO_VBUS")
-	(net 61 "unconnected-(A1-GPIO18-Pad24)")
-	(net 62 "unconnected-(A1-GPIO17-Pad22)")
-	(net 63 "unconnected-(A1-GPIO19-Pad25)")
+	(net 54 "unconnected-(U5-NC-Pad3)")
+	(net 55 "unconnected-(U5-EN-Pad5)")
+	(net 56 "LED_DIN")
+	(net 57 "unconnected-(U5-NC-Pad2)")
+	(net 58 "LED_DOUT")
+	(net 59 "PICO_VBUS")
+	(net 60 "unconnected-(A1-GPIO18-Pad24)")
+	(net 61 "unconnected-(A1-GPIO17-Pad22)")
+	(net 62 "unconnected-(A1-GPIO19-Pad25)")
 	(footprint "Capacitor_SMD:C_0402_1005Metric"
 		(layer "F.Cu")
@@
 			(layers "F.Cu" "F.Mask" "F.Paste")
 			(roundrect_rratio 0.25)
-			(net 60 "PICO_VBUS")
+			(net 59 "PICO_VBUS")
 			(pinfunction "G")
 			(pintype "input")
@@
 			(size 1.55 0.6)
 			(layers "F.Cu" "F.Mask" "F.Paste")
-			(net 58 "unconnected-(U5-NC-Pad2)")
+			(net 57 "unconnected-(U5-NC-Pad2)")
 			(pinfunction "NC")
 			(pintype "no_connect")
@@
 			(size 1.55 0.6)
 			(layers "F.Cu" "F.Mask" "F.Paste")
-			(net 55 "unconnected-(U5-NC-Pad3)")
+			(net 54 "unconnected-(U5-NC-Pad3)")
 			(pinfunction "NC")
 			(pintype "no_connect")
@@
 			(size 1.55 0.6)
 			(layers "F.Cu" "F.Mask" "F.Paste")
-			(net 56 "unconnected-(U5-EN-Pad5)")
+			(net 55 "unconnected-(U5-EN-Pad5)")
 			(pinfunction "EN")
 			(pintype "input+no_connect")
@@
 			(size 1 1)
 			(layers "F.Cu" "F.Mask")
-			(net 59 "LED_DOUT")
+			(net 58 "LED_DOUT")
 			(pinfunction "1")
 			(pintype "passive")
@@
 			(size 0.7 0.7)
 			(layers "F.Cu" "F.Mask" "F.Paste")
-			(net 57 "LED_DIN")
+			(net 56 "LED_DIN")
 			(pinfunction "DIN")
 			(pintype "input")
@@
 			(size 0.7 0.7)
 			(layers "F.Cu" "F.Mask" "F.Paste")
-			(net 59 "LED_DOUT")
+			(net 58 "LED_DOUT")
 			(pinfunction "DOUT")
 			(pintype "output")
@@
 			(layers "F.Cu" "F.Mask")
 			(roundrect_rratio 0.5)
-			(net 57 "LED_DIN")
+			(net 56 "LED_DIN")
 			(pinfunction "GPIO6")
 			(pintype "bidirectional")
@@
 			(layers "F.Cu" "F.Mask")
 			(roundrect_rratio 0.5)
-			(net 62 "unconnected-(A1-GPIO17-Pad22)")
+			(net 61 "unconnected-(A1-GPIO17-Pad22)")
 			(pinfunction "GPIO17")
 			(pintype "bidirectional+no_connect")
@@
 			(layers "F.Cu" "F.Mask")
 			(roundrect_rratio 0.5)
-			(net 61 "unconnected-(A1-GPIO18-Pad24)")
+			(net 60 "unconnected-(A1-GPIO18-Pad24)")
 			(pinfunction "GPIO18")
 			(pintype "bidirectional+no_connect")
@@
 			(layers "F.Cu" "F.Mask")
 			(roundrect_rratio 0.5)
-			(net 63 "unconnected-(A1-GPIO19-Pad25)")
+			(net 62 "unconnected-(A1-GPIO19-Pad25)")
 			(pinfunction "GPIO19")
 			(pintype "bidirectional+no_connect")
@@
 			(layers "F.Cu" "F.Mask")
 			(roundrect_rratio 0.5)
-			(net 60 "PICO_VBUS")
+			(net 59 "PICO_VBUS")
 			(pinfunction "VBUS")
 			(pintype "power_out")
@@
 		(tags "resistor")
 		(property "Reference" "R4"
-			(at -0.5 1.5 0)
+			(at -1 1.5 0)
 			(layer "F.SilkS")
 			(effects
@@
 	(footprint "Resistor_SMD:R_0402_1005Metric"
 		(layer "F.Cu")
-		(at 115.5 80 180)
+		(at 117.5 79 180)
 		(descr "Resistor SMD 0402 (1005 Metric), square (rectangular) end terminal, IPC-7351 nominal, (Body size source: IPC-SM-782 page 72, https://www.pcb-3d.com/wordpress/wp-content/uploads/ipc-sm-782a_amendment_1_and_2.pdf), generated with kicad-footprint-generator")
 		(tags "resistor")
 		(property "Reference" "R6"
-			(at 0.5 1.5 0)
+			(at 2 0.5 0)
 			(layer "F.SilkS")
 			(effects
@@
 			)
 		)
-		(property "Value" "2k2"
+		(property "Value" "100k"
 			(at 0 1.17 0)
 			(layer "F.Fab")
@@
 			)
 		)
-		(property "LCSC Part" "C25879"
+		(property "LCSC Part" "C25741"
 			(at 0 0 180)
 			(unlocked yes)
@@
 			(layers "F.Cu" "F.Mask" "F.Paste")
 			(roundrect_rratio 0.25)
-			(net 54 "Net-(R5-Pad2)")
+			(net 52 "Net-(U5-VSENSE)")
 			(pintype "passive")
 		)
@@
 		(tags "resistor")
 		(property "Reference" "R5"
-			(at 0 1.5 0)
+			(at 2 0 0)
 			(layer "F.SilkS")
 			(effects
@@
 			)
 		)
-		(property "Value" "1k"
+		(property "Value" "3k3"
 			(at 0 1.17 0)
 			(layer "F.Fab")
@@
 			)
 		)
-		(property "LCSC Part" "C11702"
+		(property "LCSC Part" "C25890"
 			(at 0 0 180)
 			(unlocked yes)
@@
 			(layers "F.Cu" "F.Mask" "F.Paste")
 			(roundrect_rratio 0.25)
-			(net 54 "Net-(R5-Pad2)")
+			(net 2 "GND")
 			(pintype "passive")
 		)
@@
 	)
 	(segment
+		(start 116.99 79)
+		(end 116.99 80)
+		(width 0.4)
+		(layer "F.Cu")
+		(net 2)
+	)
+	(segment
 		(start 124.5 112)
 		(end 124.751 112.251)
@@
 	)
 	(segment
+		(start 112.3 87.865)
+		(end 114.335 87.865)
+		(width 0.6)
+		(layer "F.Cu")
+		(net 2)
+	)
+	(segment
 		(start 127.5 111.48)
 		(end 128.02 112)
@@
 	)
 	(segment
+		(start 114.335 87.865)
+		(end 114.4 87.8)
+		(width 0.6)
+		(layer "F.Cu")
+		(net 2)
+	)
+	(segment
 		(start 128.02 112)
 		(end 127.5 112.52)
@@
 	)
 	(segment
-		(start 118.99 79.49)
-		(end 118.5 79)
+		(start 119 79)
+		(end 119 79.99)
 		(width 0.4)
 		(layer "F.Cu")
@@
 	)
 	(segment
-		(start 118.99 80)
-		(end 118.99 79.49)
+		(start 118.01 79)
+		(end 119 79)
+		(width 0.4)
+		(layer "F.Cu")
+		(net 52)
+	)
+	(segment
+		(start 118.01 79)
+		(end 118.01 80)
+		(width 0.4)
+		(layer "F.Cu")
+		(net 52)
+	)
+	(segment
+		(start 119 79.99)
+		(end 118.99 80)
 		(width 0.4)
 		(layer "F.Cu")
@@
 	)
 	(via
-		(at 118.5 79)
+		(at 119 79)
 		(size 0.6)
 		(drill 0.3)
@@
 	)
 	(segment
-		(start 119 79.5)
-		(end 118.5 79)
-		(width 0.4)
-		(layer "B.Cu")
-		(net 52)
-	)
-	(segment
 		(start 119 86.5)
-		(end 119 79.5)
+		(end 119 79)
 		(width 0.4)
 		(layer "B.Cu")
@@
 	)
 	(segment
-		(start 116.01 80)
-		(end 116.99 80)
-		(width 0.4)
-		(layer "F.Cu")
-		(net 54)
-	)
-	(segment
 		(start 125.085 102.085)
 		(end 126.099 103.099)
 		(width 0.4)
 		(layer "F.Cu")
-		(net 57)
+		(net 56)
 	)
 	(segment
@@
 		(width 0.4)
 		(layer "F.Cu")
-		(net 57)
+		(net 56)
 	)
 	(segment
@@
 		(width 0.4)
 		(layer "F.Cu")
-		(net 57)
+		(net 56)
 	)
 	(segment
@@
 		(width 0.4)
 		(layer "F.Cu")
-		(net 57)
+		(net 56)
 	)
 	(segment
@@
 		(width 0.4)
 		(layer "F.Cu")
-		(net 57)
+		(net 56)
 	)
 	(segment
@@
 		(width 0.4)
 		(layer "F.Cu")
-		(net 57)
+		(net 56)
 	)
 	(segment
@@
 		(width 0.4)
 		(layer "F.Cu")
-		(net 57)
+		(net 56)
 	)
 	(segment
@@
 		(width 0.6)
 		(layer "F.Cu")
-		(net 59)
+		(net 58)
 	)
 	(segment
@@
 		(width 0.6)
 		(layer "F.Cu")
-		(net 59)
+		(net 58)
 	)
 	(segment
@@
 		(width 0.6)
 		(layer "F.Cu")
-		(net 59)
+		(net 58)
 	)
 	(segment
@@
 		(width 0.4)
 		(layer "F.Cu")
-		(net 60)
+		(net 59)
 	)
 	(segment
@@
 		(width 0.4)
 		(layer "F.Cu")
-		(net 60)
+		(net 59)
 	)
 	(segment
@@
 		(width 0.4)
 		(layer "F.Cu")
-		(net 60)
+		(net 59)
 	)
 	(segment
@@
 		(width 0.4)
 		(layer "F.Cu")
-		(net 60)
+		(net 59)
 	)
 	(segment
@@
 		(width 0.4)
 		(layer "F.Cu")
-		(net 60)
+		(net 59)
 	)
 	(segment
@@
 		(width 0.4)
 		(layer "F.Cu")
-		(net 60)
+		(net 59)
 	)
 	(segment
@@
 		(width 0.4)
 		(layer "F.Cu")
-		(net 60)
+		(net 59)
 	)
 	(segment
@@
 		(width 0.4)
 		(layer "F.Cu")
-		(net 60)
+		(net 59)
 	)
 	(segment
@@
 		(width 0.4)
 		(layer "F.Cu")
-		(net 60)
+		(net 59)
 	)
 	(via
@@
 		(drill 0.3)
 		(layers "F.Cu" "B.Cu")
-		(net 60)
+		(net 59)
 	)
 	(via
@@
 		(drill 0.3)
 		(layers "F.Cu" "B.Cu")
-		(net 60)
+		(net 59)
 	)
 	(segment
@@
 		(width 0.4)
 		(layer "B.Cu")
-		(net 60)
+		(net 59)
 	)
 	(segment
@@
 		(width 0.4)
 		(layer "B.Cu")
-		(net 60)
+		(net 59)
 	)
 	(zone
@@
 		(polygon
 			(pts
-				(xy 120 87) (xy 125 87) (xy 125 80) (xy 124.5 79.5) (xy 120 79.5) (xy 119.5 80) (xy 119.5 86.5)
+				(xy 121 87) (xy 125 87) (xy 125 80) (xy 124.5 79.5) (xy 120 79.5) (xy 119.5 80) (xy 119.5 85.5)
 			)
 		)

Commit message: board rc3
Parts:
- removed D2, D4: WS2812B-2020, LED_SMD:LED_WS2812B-2020_PLCC4_2.0x2.0mm
- removed TP2, TP3, TP4: TestPoint, TestPoint:TestPoint_Pad_D1.0mm
- added J2: Conn_01x03, Connector_PinHeader_2.54mm:PinHeader_1x03_P2.54mm_Vertical, F.Cu at (111.5, 101.5)
- D1, D3: value WS2812B-2020 -> WS2812B; footprint LED_SMD:LED_WS2812B-2020_PLCC4_2.0x2.0mm -> LED_SMD:LED_WS2812B_PLCC4_5.0x5.0mm_P3.2mm
- moved C14 3.05 mm to (130.0, 102.5)
- moved D3 1.12 mm to (117.0, 102.5), turned to 0 degrees
- moved D1 0.71 mm to (124.5, 102.5), turned to 0 degrees
Connections:
- D1 pad 1: Net-(D1-DOUT) -> PICO_VSYS
- D1 pad 2: GND -> Net-(D1-DOUT)
- D1 pad 3: LED_DIN -> GND
- D1 pad 4: PICO_VSYS -> LED_DIN
- D3 pad 1: Net-(D3-DOUT) -> PICO_VSYS
- D3 pad 2: GND -> Net-(D3-DOUT)
- D3 pad 3: Net-(D2-DOUT) -> GND
- D3 pad 4: PICO_VSYS -> Net-(D1-DOUT)
Routing:
- net PICO_VSYS: track 112.6 -> 98.2 mm, vias 9 -> 8
- net LED_DIN: track 26.4 -> 19.9 mm
- net GND: track 63.4 -> 57.4 mm, vias 41 -> 39
- net Net-(D2-DOUT): track 3.66 -> 0.00 mm
- net LED_DOUT: track 2.84 -> 0.00 mm
- net Net-(D3-DOUT): track 3.66 -> 5.47 mm
- net DRVNSLEEP: track 59.6 -> 58.7 mm
- net Net-(D1-DOUT): track 3.66 -> 4.38 mm
- net DRVOUT2B: track 3.75 -> 4.43 mm
Other:
- board text added: "GND 5V DO"

Commit message: board rc4
Routing:
- net Net-(D6-K): track 24.8 -> 19.7 mm
- net GND: track 57.4 -> 57.8 mm, vias 39 -> 46
Changed lines of the file:
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@@
 		(tags "capacitor")
 		(property "Reference" "C13"
-			(at 3.5 0 0)
+			(at -3.5 0 0)
 			(layer "F.SilkS")
 			(effects
@@
 		(tags "capacitor")
 		(property "Reference" "C12"
-			(at 3 0 0)
+			(at 4.5 0 0)
 			(layer "F.SilkS")
 			(effects
@@
 	)
 	(segment
+		(start 110.54 112.54)
+		(end 110 112)
+		(width 0.6)
+		(layer "F.Cu")
+		(net 2)
+	)
+	(segment
 		(start 124 112)
 		(end 122.52 112)
@@
 	)
 	(segment
+		(start 111 111.48)
+		(end 110.52 111.48)
+		(width 0.6)
+		(layer "F.Cu")
+		(net 2)
+	)
+	(segment
 		(start 113 112)
 		(end 113.5 112)
@@
 	)
 	(segment
+		(start 111 112.54)
+		(end 110.54 112.54)
+		(width 0.6)
+		(layer "F.Cu")
+		(net 2)
+	)
+	(segment
 		(start 124.5 112)
 		(end 124.751 112.251)
@@
 	)
 	(segment
-		(start 110.02 111.48)
-		(end 110 111.5)
-		(width 0.6)
-		(layer "F.Cu")
-		(net 2)
-	)
-	(segment
 		(start 126.52 111.48)
 		(end 127.5 111.48)
@@
 	)
 	(segment
-		(start 110.04 112.54)
-		(end 110 112.5)
-		(width 0.6)
-		(layer "F.Cu")
-		(net 2)
-	)
-	(segment
 		(start 112.16 106.54)
 		(end 111.5 106.54)
@@
 	)
 	(segment
-		(start 110.02 111.48)
-		(end 111 111.48)
+		(start 110.52 111.48)
+		(end 110 112)
 		(width 0.6)
 		(layer "F.Cu")
@@
 	)
 	(segment
-		(start 111 112.54)
-		(end 110.04 112.54)
-		(width 0.6)
-		(layer "F.Cu")
-		(net 2)
-	)
-	(segment
 		(start 116.5 112.54)
 		(end 115.54 112.54)
@@
 	)
 	(via
-		(at 129.5 90.5)
+		(at 128.5 91.5)
+		(size 0.6)
+		(drill 0.3)
+		(layers "F.Cu" "B.Cu")
+		(free yes)
+		(net 2)
+	)
+	(via
+		(at 108.5 77.5)
 		(size 0.6)
 		(drill 0.3)
@@
 	)
 	(via
+		(at 128.5 89)
+		(size 0.6)
+		(drill 0.3)
+		(layers "F.Cu" "B.Cu")
+		(free yes)
+		(net 2)
+	)
+	(via
 		(at 148.5 101.5)
 		(size 0.6)
@@
 	)
 	(via
-		(at 115.5 111.5)
+		(at 143.5 91.5)
+		(size 0.6)
+		(drill 0.3)
+		(layers "F.Cu" "B.Cu")
+		(free yes)
+		(net 2)
+	)
+	(via
+		(at 115 112)
 		(size 0.6)
 		(drill 0.3)
@@
 	)
 	(via
+		(at 116.5 84.5)
+		(size 0.6)
+		(drill 0.3)
+		(layers "F.Cu" "B.Cu")
+		(free yes)
+		(net 2)
+	)
+	(via
 		(at 134.5 96.5)
 		(size 0.6)
@@
 	)
 	(via
-		(at 124 98.5)
+		(at 131.5 113)
 		(size 0.6)
 		(drill 0.3)
@@
 	)
 	(via
-		(at 130 86.5)
+		(at 124 98.5)
 		(size 0.6)
 		(drill 0.3)
@@
 	)
 	(via
-		(at 134 117.5)
+		(at 149.5 83.5)
 		(size 0.6)
 		(drill 0.3)
@@
 	)
 	(via
-		(at 124.5 104)
+		(at 128.5 86.5)
 		(size 0.6)
 		(drill 0.3)
@@
 	)
 	(via
-		(at 141 71.5)
+		(at 134 117.5)
 		(size 0.6)
 		(drill 0.3)
@@
 	)
 	(via
-		(at 121 111.5)
+		(at 124.5 104)
 		(size 0.6)
 		(drill 0.3)
 		(layers "F.Cu" "B.Cu")
+		(free yes)
 		(net 2)
 	)
 	(via
-		(at 114 81.5)
+		(at 141 71.5)
 		(size 0.6)
 		(drill 0.3)
@@
 	)
 	(via
-		(at 115.5 112.5)
+		(at 120.5 112)
 		(size 0.6)
 		(drill 0.3)
@@
 	)
 	(via
+		(at 116.5 81.5)
+		(size 0.6)
+		(drill 0.3)
+		(layers "F.Cu" "B.Cu")
+		(free yes)
+		(net 2)
+	)
+	(via
 		(at 108 117.5)
 		(size 0.6)
@@
 	)
 	(via
+		(at 109 112)
+		(size 0.6)
+		(drill 0.3)
+		(layers "F.Cu" "B.Cu")
+		(net 2)
+	)
+	(via
 		(at 116 98.5)
 		(size 0.6)
@@
 	)
 	(via
-		(at 121.02 112.52)
+		(at 115 84.5)
 		(size 0.6)
 		(drill 0.3)
 		(layers "F.Cu" "B.Cu")
+		(free yes)
 		(net 2)
 	)
@@
 	)
 	(via
-		(at 114 83)
+		(at 116.5 83)
+		(size 0.6)
+		(drill 0.3)
+		(layers "F.Cu" "B.Cu")
+		(free yes)
+		(net 2)
+	)
+	(via
+		(at 115 83)
 		(size 0.6)
 		(drill 0.3)
@@
 	)
 	(via
-		(at 112.5 83)
+		(at 133.5 84)
 		(size 0.6)
 		(drill 0.3)
@@
 	)
 	(via
-		(at 112.5 81.5)
+		(at 115 81.5)
 		(size 0.6)
 		(drill 0.3)
@@
 	)
 	(via
-		(at 128.5 105)
+		(at 126.5 84.5)
 		(size 0.6)
 		(drill 0.3)
@@
 	)
 	(via
-		(at 103.5 77.5)
+		(at 128.5 105)
 		(size 0.6)
 		(drill 0.3)
@@
 	)
 	(via
-		(at 110 111.5)
+		(at 103.5 77.5)
 		(size 0.6)
 		(drill 0.3)
 		(layers "F.Cu" "B.Cu")
+		(free yes)
 		(net 2)
 	)
 	(via
-		(at 126.52 111.48)
+		(at 110 112)
 		(size 0.6)
 		(drill 0.3)
@@
 	)
 	(via
-		(at 110.04 112.54)
+		(at 126.52 111.48)
 		(size 0.6)
 		(drill 0.3)
@@
 	)
 	(segment
-		(start 122 96.5)
-		(end 123 95.5)
-		(width 2)
-		(layer "F.Cu")
-		(net 23)
-	)
-	(segment
-		(start 119 96.5)
-		(end 122 96.5)
-		(width 2)
-		(layer "F.Cu")
-		(net 23)
-	)
-	(segment
-		(start 113 96.5)
-		(end 117 96.5)
-		(width 2)
-		(layer "F.Cu")
-		(net 23)
-	)
-	(segment
 		(start 112.3 90.405)
 		(end 112.3 92.7)
@@
 	)
 	(segment
-		(start 123 95.5)
+		(start 121.025 95.5)
 		(end 123 93.525)
-		(width 2)
-		(layer "F.Cu")
-		(net 23)
-	)
-	(segment
-		(start 111.5 95)
-		(end 113 96.5)
-		(width 2)
-		(layer "F.Cu")
-		(net 23)
-	)
-	(segment
-		(start 118 95.5)
-		(end 117 96.5)
-		(width 0.6)
+		(width 1.6)
 		(layer "F.Cu")
 		(net 23)
@@
 	)
 	(segment
-		(start 118 95.5)
-		(end 119 96.5)
-		(width 0.6)
+		(start 112.3 92.7)
+		(end 111.5 93.5)
+		(width 1)
 		(layer "F.Cu")
 		(net 23)
 	)
 	(segment
-		(start 112.3 92.7)
-		(end 111.5 93.5)
-		(width 1)
+		(start 111.5 93.5)
+		(end 111.5 94.5)
+		(width 1.6)
 		(layer "F.Cu")
 		(net 23)
 	)
 	(segment
-		(start 117 96.5)
-		(end 119 96.5)
-		(width 2)
+		(start 111.5 94.5)
+		(end 112.5 95.5)
+		(width 1.6)
 		(layer "F.Cu")
 		(net 23)
 	)
 	(segment
-		(start 111.5 93.5)
-		(end 111.5 95)
-		(width 2)
+		(start 112.5 95.5)
+		(end 121.025 95.5)
+		(width 1.6)
 		(layer "F.Cu")
 		(net 23)
@@
 		(polygon
 			(pts
-				(xy 100 64) (xy 100 115.5) (xy 128.5 115.5) (xy 128.5 112.5) (xy 108.5 112.5) (xy 108.5 105.5) (xy 112.5 105.5)
-				(xy 112.5 96) (xy 125 83) (xy 125 73.5) (xy 137 73.5) (xy 137 64)
+				(xy 100 64) (xy 100 115.5) (xy 128.5 115.5) (xy 128.5 112.5) (xy 108.5 112.5) (xy 108.5 105) (xy 112.5 105)
+				(xy 112.5 97) (xy 125 84) (xy 125 73.5) (xy 137 73.5) (xy 137 64)
+			)
+		)
+	)
+	(zone
+		(net 2)
+		(net_name "GND")
+		(layer "In2.Cu")
+		(hatch edge 0.5)
+		(priority 4)
+		(connect_pads
+			(clearance 0.6)
+		)
+		(min_thickness 0.25)
+		(filled_areas_thickness no)
+		(fill yes
+			(thermal_gap 0.5)
+			(thermal_bridge_width 0.5)
+		)
+		(polygon
+			(pts
+				(xy 117 81) (xy 114.5 81) (xy 114 81.5) (xy 114 90) (xy 114.5 90.5) (xy 115.5 90.5) (xy 116 90)
+				(xy 116 86) (xy 117.5 84.5) (xy 117.5 81.5)
 			)
 		)

Commit message: board rc5
Routing:
- net GND: track 57.8 -> 22.4 mm, vias 46 -> 45
- net +3V3: track 137.1 -> 137.7 mm
