File: pcb/rp2040-board.kicad_sch (KiCad schematic)
At the start: 51 parts, among them J1 DMX, J2 GPIO, J3 ELRS, J4 OLED, J5 Conn_ARM_JTAG_SWD_10, J6 USB_C_Receptacle_USB2.0_16P, SW1 USB Boot, SW2 RotaryEncoder_Switch, SW3 Reset, U1 W25Q128JVS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

Commit message: board wip
Parts:
- J2: footprint Connector_PinHeader_2.54mm:PinHeader_1x26_P2.54mm_Vertical -> Connector_PinHeader_2.54mm:PinHeader_1x22_P2.54mm_Vertical; symbol Connector_Generic:Conn_01x26 -> Connector_Generic:Conn_01x22
- J5: value Conn_ARM_JTAG_SWD_10 -> SWD
Connections:
- net +3V3: now also J2.2 (Pin_2)
- net +5V: now also J2.1 (Pin_1)
- net GND: now also J2.13 (Pin_13), J2.22 (Pin_22), J2.3 (Pin_3), J2.4 (Pin_4)
- net GPIO05: now reaches J2.10 (Pin_10)
- net GPIO05: now also U3.7 (GPIO5)
- net GPIO06: now reaches J2.11 (Pin_11)
- net GPIO06: now also U3.8 (GPIO6)
- net GPIO07: now reaches J2.12 (Pin_12)
- net GPIO07: now also U3.9 (GPIO7)
- net GPIO08: now reaches J2.14 (Pin_14)
- net GPIO08: now also U3.11 (GPIO8)
- net GPIO09: now reaches J2.15 (Pin_15)
- net GPIO09: now also U3.12 (GPIO9)
- net GPIO10: now reaches J2.16 (Pin_16)
- net GPIO10: now also U3.13 (GPIO10)
- net GPIO11: now reaches J2.17 (Pin_17)
- net GPIO11: now also U3.14 (GPIO11)
- net GPIO12: now reaches J2.18 (Pin_18)
- net GPIO12: now also U3.15 (GPIO12)
- net GPIO13: now reaches J2.19 (Pin_19)
- net GPIO13: now also U3.16 (GPIO13)
- net GPIO14: now reaches J2.20 (Pin_20)
- net GPIO14: now also U3.17 (GPIO14)
- net GPIO15: now reaches J2.21 (Pin_21)
- net GPIO15: now also U3.18 (GPIO15)
- net GPIO00: now reaches J2.5 (Pin_5)
- net GPIO00: now also U3.2 (GPIO0)
- net GPIO01: now reaches J2.6 (Pin_6)
- net GPIO01: now also U3.3 (GPIO1)
- net GPIO02: now reaches J2.7 (Pin_7)
- net GPIO02: now also U3.4 (GPIO2)
- net GPIO03: now reaches J2.8 (Pin_8)
- net GPIO03: now also U3.5 (GPIO3)
- net GPIO04: now reaches J2.9 (Pin_9)
- net GPIO04: now also U3.6 (GPIO4)
Other:
- moved on the sheet: J3

Commit message: board wip
Connections:
- net LED_D1: now also U3.28 (GPIO17); no longer U3.37 (GPIO25)
- net LED_D2: now also U3.29 (GPIO18); no longer U3.36 (GPIO24)
- net OLED_SCK: now also U3.37 (GPIO25); no longer U3.28 (GPIO17)
- net OLED_SDA: now also U3.36 (GPIO24); no longer U3.29 (GPIO18)
Changed lines of the file:
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@@
     )
   )
-  (global_label "LED_D1" (shape input) (at 154.94 110.49 0) (fields_autoplaced)
-    (effects (font (size 1.27 1.27)) (justify left))
-    (property "Intersheetrefs" "${INTERSHEET_REFS}" (at 164.8194 110.49 0)
+  (global_label "LED_D1" (shape input) (at 154.94 90.17 0) (fields_autoplaced)
+    (effects (font (size 1.27 1.27)) (justify left))
+    (property "Intersheetrefs" "${INTERSHEET_REFS}" (at 164.8194 90.17 0)
       (effects (font (size 1.27 1.27)) (justify left) hide)
     )
@@
     )
   )
-  (global_label "OLED_SDA" (shape input) (at 154.94 92.71 0) (fields_autoplaced)
-    (effects (font (size 1.27 1.27)) (justify left))
-    (property "Intersheetrefs" "${INTERSHEET_REFS}" (at 167.2385 92.71 0)
+  (global_label "OLED_SDA" (shape input) (at 154.94 107.95 0) (fields_autoplaced)
+    (effects (font (size 1.27 1.27)) (justify left))
+    (property "Intersheetrefs" "${INTERSHEET_REFS}" (at 167.2385 107.95 0)
       (effects (font (size 1.27 1.27)) (justify left) hide)
     )
@@
     )
   )
-  (global_label "OLED_SCK" (shape input) (at 154.94 90.17 0) (fields_autoplaced)
-    (effects (font (size 1.27 1.27)) (justify left))
-    (property "Intersheetrefs" "${INTERSHEET_REFS}" (at 167.4199 90.17 0)
+  (global_label "OLED_SCK" (shape input) (at 154.94 110.49 0) (fields_autoplaced)
+    (effects (font (size 1.27 1.27)) (justify left))
+    (property "Intersheetrefs" "${INTERSHEET_REFS}" (at 167.4199 110.49 0)
       (effects (font (size 1.27 1.27)) (justify left) hide)
     )
@@
     )
   )
-  (global_label "LED_D2" (shape input) (at 154.94 107.95 0) (fields_autoplaced)
-    (effects (font (size 1.27 1.27)) (justify left))
-    (property "Intersheetrefs" "${INTERSHEET_REFS}" (at 164.8194 107.95 0)
-      (effects (font (size 1.27 1.27)) (justify left) hide)
-    )
+  (global_label "LED_D2" (shape input) (at 154.94 92.71 0) (fields_autoplaced)
+    (effects (font (size 1.27 1.27)) (justify left))
+    (property "Intersheetrefs" "${INTERSHEET_REFS}" (at 164.8194 92.71 0)
+      (effects (font (size 1.27 1.27)) (justify left) hide)
+    )

Commit message: board wip
Parts:
- R11: footprint Resistor_SMD:R_0402_1005Metric -> Resistor_SMD:R_0603_1608Metric; LCSC Part C17168 -> C21189
Connections:
- net +3V3: now also J2.3 (Pin_3); no longer J2.2 (Pin_2)
- net +5V: now also J2.2 (Pin_2); no longer J2.1 (Pin_1)
- net GND: no longer J2.3 (Pin_3)
- net RS485_RE_NDE: now also U3.39 (GPIO27_ADC1)
- net RS485_RXD: now also U3.40 (GPIO28_ADC2)
- net RS485_TXD: now also U3.38 (GPIO26_ADC0)
- net VBUS: now also J2.1 (Pin_1)
- net USB_DM renamed USB_D-
- net USB_DP renamed USB_D+
Other:
- moved on the sheet: J2, J3, J4

Commit message: board rc1
Connections:
- no-connect marks 5 -> 6
Changed lines of the file:
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@@
   (no_connect (at 49.53 177.8))
   (no_connect (at 49.53 157.48))
+  (no_connect (at 154.94 123.19))
   (no_connect (at 49.53 154.94))
   (no_connect (at 49.53 180.34))

Commit message: board rc2
Changed lines of the file:
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@@
     (stroke (width 0) (type default))
   )
+  (wire (pts (xy 68.58 147.32) (xy 68.58 149.86))
+    (stroke (width 0) (type default))
+  )
   (wire (pts (xy 68.58 149.86) (xy 80.01 149.86))
     (stroke (width 0) (type default))
@@
     )
   )
+  (symbol (lib_id "power:PWR_FLAG") (at 68.58 147.32 0) (unit 1)
+    (in_bom yes) (on_board yes) (dnp no) (fields_autoplaced)
+    (property "Reference" "#FLG01" (at 68.58 145.415 0)
+      (effects (font (size 1.27 1.27)) hide)
+    )
+    (property "Value" "PWR_FLAG" (at 68.58 142.24 0)
+      (effects (font (size 1.27 1.27)))
+    )
+    (property "Footprint" "" (at 68.58 147.32 0)
+      (effects (font (size 1.27 1.27)) hide)
+    )
+    (property "Datasheet" "~" (at 68.58 147.32 0)
+      (effects (font (size 1.27 1.27)) hide)
+    )
+    (pin "1")
+    (instances
+      (project "rp2040-board"
+        (path "/75fe2d07-4ff9-4014-b967-9ecbb30e480e"
+          (reference "#FLG01") (unit 1)
+        )
+      )
+    )
+  )
   (symbol (lib_id "Interface_UART:MAX485E") (at 218.44 143.51 0) (unit 1)
     (in_bom yes) (on_board yes) (dnp no)
@@
     )
   )
+  (symbol (lib_id "power:PWR_FLAG") (at 68.58 170.18 0) (unit 1)
+    (in_bom yes) (on_board yes) (dnp no) (fields_autoplaced)
+    (property "Reference" "#FLG02" (at 68.58 168.275 0)
+      (effects (font (size 1.27 1.27)) hide)
+    )
+    (property "Value" "PWR_FLAG" (at 68.58 165.1 0)
+      (effects (font (size 1.27 1.27)))
+    )
+    (property "Footprint" "" (at 68.58 170.18 0)
+      (effects (font (size 1.27 1.27)) hide)
+    )
+    (property "Datasheet" "~" (at 68.58 170.18 0)
+      (effects (font (size 1.27 1.27)) hide)
+    )
+    (pin "1")
+    (instances
+      (project "rp2040-board"
+        (path "/75fe2d07-4ff9-4014-b967-9ecbb30e480e"
+          (reference "#FLG02") (unit 1)
+        )
+      )
+    )
+  )
   (symbol (lib_id "power:GND") (at 93.98 99.06 0) (unit 1)
     (in_bom yes) (on_board yes) (dnp no) (fields_autoplaced)
@@
         )
       )
+    )
+  )
+  (symbol (lib_id "power:GND") (at 68.58 170.18 0) (unit 1)
+    (in_bom yes) (on_board yes) (dnp no) (fields_autoplaced)
+    (property "Reference" "#PWR053" (at 68.58 176.53 0)
+      (effects (font (size 1.27 1.27)) hide)
+    )
+    (property "Value" "GND" (at 68.58 175.26 0)
+      (effects (font (size 1.27 1.27)) hide)
+    )
+    (property "Footprint" "" (at 68.58 170.18 0)
+      (effects (font (size 1.27 1.27)) hide)
+    )
+    (property "Datasheet" "" (at 68.58 170.18 0)
+      (effects (font (size 1.27 1.27)) hide)
+    )
+    (pin "1")
+    (instances
+      (project "rp2040-board"
+        (path "/75fe2d07-4ff9-4014-b967-9ecbb30e480e"
+          (reference "#PWR053") (unit 1)
+        )
+      )

Commit message: board rc3
Parts:
- added C20, C21: 4.7n, Capacitor_SMD:C_0402_1005Metric, symbol Device:C
- added C22: 22u, Capacitor_SMD:C_0805_2012Metric, symbol Device:C
- added C23: 100n, Capacitor_SMD:C_0402_1005Metric, symbol Device:C
- added C24: 1u, Capacitor_SMD:C_0402_1005Metric, symbol Device:C
- added J7: AUDIO, Connector_PinHeader_2.54mm:PinHeader_1x02_P2.54mm_Vertical, symbol Connector_Generic:Conn_01x02
- added R14, R15: 1k5, Resistor_SMD:R_0402_1005Metric, symbol Device:R
- added R16: 0, Resistor_SMD:R_0603_1608Metric, symbol Device:R
- added U5: OP07CDR, Package_SO:SOIC-8_3.9x4.9mm_P1.27mm, symbol Amplifier_Operational:OP07
Connections:
- net +5V: now also R16.2
- net GND: now also C20.2, C23.2, C24.2, J7.2 (Pin_2), U5.4 (V-)
- net PWM_AUDIO: now reaches U3.41 (GPIO29_ADC3)
- net PWM_AUDIO: now also R15.1
- new net: C21.1, R14.1, R15.2
- new net: C21.2, C22.1, U5.2 (-), U5.6
- new net: C22.2, J7.1 (Pin_1)
- new net: C20.1, R14.2, U5.3 (+)
- new net: C23.1, C24.1, R16.1, U5.7 (V+)
- no-connect marks 6 -> 7
Other:
- moved on the sheet: J2, J3, J4

Commit message: board rc4, BOM cleanup
Parts:
- J1, J2, J3, J4, J5, J7, R1, SW2: JLCPCB BOM (none) -> false
- SW1: value USB Boot -> TS-1187A-B-A-B
- SW3: value Reset -> TS-1187A-B-A-B
Other:
- note added: "Reset"
- note added: "USB Boot"

Commit message: enlarge power supply caps
Parts:
- C18, C19: value 10u -> 22u; footprint Capacitor_SMD:C_0603_1608Metric -> Capacitor_SMD:C_0805_2012Metric; LCSC Part C19702 -> C45783
Changed lines of the file:
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@@
       (effects (font (size 1.27 1.27)) (justify left))
     )
-    (property "Value" "10u" (at 104.14 157.48 0)
-      (effects (font (size 1.27 1.27)) (justify left))
-    )
-    (property "Footprint" "Capacitor_SMD:C_0603_1608Metric" (at 103.8352 158.75 0)
-      (effects (font (size 1.27 1.27)) hide)
-    )
-    (property "Datasheet" "https://datasheet.lcsc.com/lcsc/2304140030_Samsung-Electro-Mechanics-CL10A106KP8NNNC_C19702.pdf" (at 102.87 154.94 0)
-      (effects (font (size 1.27 1.27)) hide)
-    )
-    (property "LCSC Part" "C19702" (at 102.87 154.94 0)
+    (property "Value" "22u" (at 104.14 157.48 0)
+      (effects (font (size 1.27 1.27)) (justify left))
+    )
+    (property "Footprint" "Capacitor_SMD:C_0805_2012Metric" (at 103.8352 158.75 0)
+      (effects (font (size 1.27 1.27)) hide)
+    )
+    (property "Datasheet" "https://datasheet.lcsc.com/lcsc/2304140030_Samsung-Electro-Mechanics-CL21A226MAQNNNE_C45783.pdf" (at 102.87 154.94 0)
+      (effects (font (size 1.27 1.27)) hide)
+    )
+    (property "LCSC Part" "C45783" (at 102.87 154.94 0)
       (effects (font (size 1.27 1.27)) hide)
     )
@@
       (effects (font (size 1.27 1.27)) (justify left))
     )
-    (property "Value" "10u" (at 81.28 157.48 0)
-      (effects (font (size 1.27 1.27)) (justify left))
-    )
-    (property "Footprint" "Capacitor_SMD:C_0603_1608Metric" (at 80.9752 158.75 0)
-      (effects (font (size 1.27 1.27)) hide)
-    )
-    (property "Datasheet" "https://datasheet.lcsc.com/lcsc/2304140030_Samsung-Electro-Mechanics-CL10A106KP8NNNC_C19702.pdf" (at 80.01 154.94 0)
-      (effects (font (size 1.27 1.27)) hide)
-    )
-    (property "LCSC Part" "C19702" (at 80.01 154.94 0)
-      (effects (font (size 1.27 1.27)) hide)
-    )
+    (property "Value" "22u" (at 81.28 157.48 0)
+      (effects (font (size 1.27 1.27)) (justify left))
+    )
+    (property "Footprint" "Capacitor_SMD:C_0805_2012Metric" (at 80.9752 158.75 0)
+      (effects (font (size 1.27 1.27)) hide)
+    )
+    (property "Datasheet" "https://datasheet.lcsc.com/lcsc/2304140030_Samsung-Electro-Mechanics-CL21A226MAQNNNE_C45783.pdf" (at 80.01 154.94 0)
+      (effects (font (size 1.27 1.27)) hide)
+    )
+    (property "LCSC Part" "C45783" (at 80.01 154.94 0)
+      (effects (font (size 1.27 1.27)) hide)
+    )
