File: pcb/motor_drivers.kicad_sch (KiCad schematic)
At the start: 12 parts, among them U5 DRV8837, U6 DRV8837, U7 DRV8837, U8 DRV8837

Commit message: WIP on the motor driver board
Parts:
- added J5: Screw_Terminal_01x08, TerminalBlock_Phoenix:TerminalBlock_Phoenix_MKDS-1,5-8-5.08_1x08_P5.08mm_Horizontal, symbol Connector:Screw_Terminal_01x08
Connections:
- net DRVOUT1A: now also J5.1 (Pin_1)
- net DRVOUT1B: now also J5.2 (Pin_2)
- net DRVOUT2A: now also J5.3 (Pin_3)
- net DRVOUT2B: now also J5.4 (Pin_4)
- net DRVOUT3A: now also J5.5 (Pin_5)
- net DRVOUT3B: now also J5.6 (Pin_6)
- net DRVOUT4A: now also J5.7 (Pin_7)
- net DRVOUT4B: now also J5.8 (Pin_8)

Commit message: wip on pcb
Parts:
- removed J5: Screw_Terminal_01x08, TerminalBlock_Phoenix:TerminalBlock_Phoenix_MKDS-1,5-8-5.08_1x08_P5.08mm_Horizontal, symbol Connector:Screw_Terminal_01x08
- added J6: Conn_01x08, Connector_PinSocket_2.54mm:PinSocket_1x08_P2.54mm_Vertical, symbol Connector_Generic:Conn_01x08
Connections:
- net DRVOUT1A: now also J6.1 (Pin_1)
- net DRVOUT1B: now also J6.2 (Pin_2)
- net DRVOUT2A: now also J6.3 (Pin_3)
- net DRVOUT2B: now also J6.4 (Pin_4)
- net DRVOUT3A: now also J6.5 (Pin_5)
- net DRVOUT3B: now also J6.6 (Pin_6)
- net DRVOUT4A: now also J6.7 (Pin_7)
- net DRVOUT4B: now also J6.8 (Pin_8)
Changed lines of the file:
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@@
+	)
+	(symbol
+		(lib_id "Connector_Generic:Conn_01x08")
+		(at 182.88 96.52 0)
+		(unit 1)
+		(exclude_from_sim no)
+		(in_bom yes)
+		(on_board yes)
+		(dnp no)
+		(fields_autoplaced yes)
+		(property "Reference" "J6"
+			(at 185.42 96.5199 0)
+			(effects
+				(font
+					(size 1.27 1.27)
+				)
+				(justify left)
+			)
+		)
+		(property "Value" "Conn_01x08"
+			(at 185.42 99.0599 0)
+			(effects
+				(font
+					(size 1.27 1.27)
+				)
+				(justify left)
+			)
+		)
+		(property "Footprint" "Connector_PinSocket_2.54mm:PinSocket_1x08_P2.54mm_Vertical"
+			(at 182.88 96.52 0)
+			(effects
+				(font
+					(size 1.27 1.27)
+				)
+				(hide yes)
+			)
+		)
+		(property "Datasheet" "~"
+			(at 182.88 96.52 0)
+			(effects
+				(font
+					(size 1.27 1.27)
+				)
+				(hide yes)
+			)
+		)
+		(property "Description" "Generic connector, single row, 01x08, script generated (kicad-library-utils/schlib/autogen/connector/)"
+			(at 182.88 96.52 0)
+			(effects
+				(font
+					(size 1.27 1.27)
+				)
+				(hide yes)
+			)
+		)
+		(pin "3"
+		)
+		(pin "7"
+		)
+		(pin "5"
+		)
+		(pin "2"
+		)
+		(pin "4"
+		)
+		(pin "8"
+		)
+		(pin "1"
+		)
+		(pin "6"
+		)
+		(instances
+			(project ""
+				(path "/75fe2d07-4ff9-4014-b967-9ecbb30e480e/77a68358-fa71-49de-9938-40fd4b662344"
+					(reference "J6")
+					(unit 1)
+				)
+			)
+		)
 	)
 	(symbol
@@
 					(unit 1)
 				)
-			)
-		)
-	)
-	(symbol
-		(lib_id "Connector:Screw_Terminal_01x08")
-		(at 182.88 96.52 0)
-		(unit 1)
-		(exclude_from_sim no)
-		(in_bom yes)
-		(on_board yes)
-		(dnp no)
-		(fields_autoplaced yes)
-		(property "Reference" "J5"
-			(at 185.42 96.5199 0)
-			(effects
-				(font
-					(size 1.27 1.27)
-				)
-				(justify left)
-			)
-		)
-		(property "Value" "Screw_Terminal_01x08"
-			(at 185.42 99.0599 0)
-			(effects
-				(font
-					(size 1.27 1.27)
-				)
-				(justify left)
-			)
-		)
-		(property "Footprint" "TerminalBlock_Phoenix:TerminalBlock_Phoenix_MKDS-1,5-8-5.08_1x08_P5.08mm_Horizontal"
-			(at 182.88 96.52 0)
-			(effects
-				(font
-					(size 1.27 1.27)
-				)
-				(hide yes)
-			)
-		)
-		(property "Datasheet" "~"
-			(at 182.88 96.52 0)
-			(effects
-				(font
-					(size 1.27 1.27)
-				)
-				(hide yes)
-			)
-		)
-		(property "Description" "Generic screw terminal, single row, 01x08, script generated (kicad-library-utils/schlib/autogen/connector/)"
-			(at 182.88 96.52 0)
-			(effects
-				(font
-					(size 1.27 1.27)
-				)
-				(hide yes)
-			)
-		)
-		(pin "5"
-		)
-		(pin "3"
-		)
-		(pin "8"
-		)
-		(pin "6"
-		)
-		(pin "2"
-		)
-		(pin "1"
-		)
-		(pin "7"
-		)
-		(pin "4"
-		)
-		(instances
-			(project ""
-				(path "/75fe2d07-4ff9-4014-b967-9ecbb30e480e/77a68358-fa71-49de-9938-40fd4b662344"
-					(reference "J5")
-					(unit 1)
-				)

Commit message: wip on the pcb
Parts:
- J4: renamed from J6; footprint Connector_PinSocket_2.54mm:PinSocket_1x08_P2.54mm_Vertical -> Connector_PinHeader_2.54mm:PinHeader_1x08_P2.54mm_Vertical
- renumbered C20 to C1, C21 to C2, C22 to C3, C23 to C4, C24 to C5, C26 to C6, C25 to C7, C27 to C8, U5 to U1, U6 to U2, U7 to U3, U8 to U4
Connections:
- net +6V renamed +5V

Commit message: board final touches
Parts:
- J4: now left out of the parts list
Changed lines of the file:
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@@
 		(unit 1)
 		(exclude_from_sim no)
-		(in_bom yes)
+		(in_bom no)
 		(on_board yes)
 		(dnp no)
