File: pcb/power.kicad_sch (KiCad schematic)
At the start: 13 parts, among them J6 USB_C_Receptacle_USB2.0_16P, J7 Raspberry_Pi_4, U4 AMS1117-3.3, U9 TPS5430DDA

Commit message: WIP on the motor driver board
Parts:
- removed C18, C19: 22u, Capacitor_SMD:C_0805_2012Metric, symbol Device:C
- removed J6: USB_C_Receptacle_USB2.0_16P, Connector_USB:USB_C_Receptacle_G-Switch_GT-USB-7010ASV, symbol Connector:USB_C_Receptacle_USB2.0_16P
- removed R11: 0, Resistor_SMD:R_0603_1608Metric, symbol Device:R
- removed U4: AMS1117-3.3, Package_TO_SOT_SMD:SOT-223, symbol Regulator_Linear:XC6206PxxxMR
- added C28: 47uF, Capacitor_SMD:C_1206_3216Metric, symbol Device:C
- added C29: 1uF, Capacitor_SMD:C_0805_2012Metric, symbol Device:C
- added J1: Input, TerminalBlock_Phoenix:TerminalBlock_Phoenix_MKDS-1,5-2-5.08_1x02_P5.08mm_Horizontal, symbol Connector:Screw_Terminal_01x02
- added R3: 1k, Resistor_SMD:R_0402_1005Metric, symbol Device:R
- added R6: 2k2, Resistor_SMD:R_0402_1005Metric, symbol Device:R
- J7: footprint (none) -> Connector_PinSocket_2.54mm:PinSocket_2x20_P2.54mm_Vertical
- L1: value L -> 15uH; footprint (none) -> Inductor_SMD:L_Changjiang_FXL0630; LCSC Part (none) -> C177243
Connections:
- net +5V: now also J7.2 (5V), J7.4 (5V), L1.2, R14.1, C28.1, C29.1; no longer D5.1 (K)
- net GND: now also C15.2, J7.14 (GND), J7.20 (GND), J7.25 (GND), J7.30 (GND), J7.34 (GND), J7.39 (GND), J7.6 (GND), J7.9 (GND), C28.2, C29.2, J1.1 (Pin_1), R6.2
- net VCC: now reaches C15.1
- net VCC: now also D5.1 (K), U9.7 (VIN), J1.2 (Pin_2)
- net at U9.4 (VSENSE): now also R14.2, R3.1
- net I2C_SDA: now reaches J7.3 (SDA_I2C1/GPIO02)
- net I2C_SCK: now reaches J7.5 (SCL_I2C1/GPIO03)
- new net: R3.2, R6.1
- no-connect marks 4 -> 2
Other:
- moved on the sheet: C14, C15, D5, D6, J7, L1, R14, U9

Commit message: wip on pcb
Parts:
- added C1: 1uF, Capacitor_SMD:C_0805_2012Metric, symbol Device:C
- added H1, H2, H3, H4: MountingHole, MountingHole:MountingHole_2.7mm, symbol Mechanical:MountingHole
Connections:
- net GND: now also C1.2
- net VCC: now also C1.1

Commit message: wip on the pcb
Parts:
- removed J1: Input, TerminalBlock_Phoenix:TerminalBlock_Phoenix_MKDS-1,5-2-5.08_1x02_P5.08mm_Horizontal, symbol Connector:Screw_Terminal_01x02
- added J5: PWR IN, Connector_AMASS:AMASS_XT30U-M_1x02_P5.0mm_Vertical, symbol Connector_Generic:Conn_01x02
- added Q1: AO3401A, Package_TO_SOT_SMD:SOT-23, symbol Transistor_FET:AO3401A
- added TP1: TestPoint, TestPoint:TestPoint_Pad_D1.0mm, symbol Connector:TestPoint
- C11: renamed from C15; value 22u -> 22uF
- C12: renamed from C28; value 47uF -> 22uF; footprint Capacitor_SMD:C_1206_3216Metric -> Capacitor_SMD:C_0805_2012Metric; LCSC Part C96123 -> C45783
- J6: renamed from J7; footprint Connector_PinSocket_2.54mm:PinSocket_2x20_P2.54mm_Vertical -> Connector_PinSocket_2.54mm:PinSocket_2x10_P2.54mm_Vertical
- renumbered C1 to C10, C29 to C13, C14 to C9, R14 to R4, R3 to R5, U9 to U5
Connections:
- net +5V: now also TP1.1
- net GND: now also J5.1 (Pin_1)
- net VCC renamed VIN
- net VIN: now also J5.2 (Pin_2), Q1.3 (D)
- new net PICO_VBUS: Q1.1 (G)
- new net PICO_VSYS: Q1.2 (S)
- no-connect marks 2 -> 28

Commit message: wip on the pcb
Parts:
- added H5, H6, H7, H8: MountingHole, MountingHole:MountingHole_2.2mm_M2, symbol Mechanical:MountingHole
Connections:
- net +5V: now also Q1.3 (D)
- net VIN: no longer Q1.3 (D)
- net RP_TX: now reaches J6.10 (GPIO15/UART_RXD)
- net RP_RX: now reaches J6.8 (GPIO14/UART_TXD)
- no-connect marks 28 -> 26
Other:
- moved on the sheet: C10, C11, C12, C13, C9, D5, D6, J5, L1, Q1, R4, R5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

Commit message: pcb almost done
Connections:
- net GPIO03: now reaches J6.13 (GPIO27/SDIO_DAT3)
- net GPIO02: now reaches J6.15 (GPIO22/SDIO_CLK)
- no-connect marks 26 -> 24
Changed lines of the file:
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@@
-	)
-	(no_connect
-		(at 196.85 67.31)
 	)
 	(no_connect
@@
 	)
 	(no_connect
-		(at 196.85 80.01)
-	)
-	(no_connect
 		(at 196.85 74.93)
 	)
@@
 		)
 	)
+	(global_label "GPIO03"
+		(shape input)
+		(at 196.85 80.01 180)
+		(fields_autoplaced yes)
+		(effects
+			(font
+				(size 1.27 1.27)
+			)
+			(justify right)
+		)
+		(property "Intersheetrefs" "${INTERSHEET_REFS}"
+			(at 186.9705 80.01 0)
+			(effects
+				(font
+					(size 1.27 1.27)
+				)
+				(justify right)
+				(hide yes)
+			)
+		)
+	)
 	(global_label "PICO_VSYS"
 		(shape input)
@@
 				(hide yes)
 			)
+		)
+	)
+	(global_label "GPIO02"
+		(shape input)
+		(at 196.85 67.31 180)
+		(fields_autoplaced yes)
+		(effects
+			(font
+				(size 1.27 1.27)
+			)
+			(justify right)
+		)
+		(property "Intersheetrefs" "${INTERSHEET_REFS}"
+			(at 186.9705 67.31 0)
+			(effects
+				(font
+					(size 1.27 1.27)
+				)
+				(justify right)
+				(hide yes)
+			)

Commit message: board final touches
Parts:
- C11: value 22uF -> 10uF; LCSC Part C45783 -> C440198
- J5, J6, TP1: now left out of the parts list
- Q1: LCSC Part (none) -> C15127
Changed lines of the file:
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@@
 			)
 		)
-		(property "Value" "22uF"
+		(property "Value" "10uF"
 			(at 66.04 52.07 0)
 			(effects
@@
 			)
 		)
-		(property "LCSC Part" "C45783"
+		(property "LCSC Part" "C440198"
 			(at 64.77 49.53 0)
 			(effects
@@
 		(unit 1)
 		(exclude_from_sim no)
-		(in_bom yes)
+		(in_bom no)
 		(on_board yes)
 		(dnp no)
@@
 			)
 		)
+		(property "LCSC Part" "C15127"
+			(at 138.43 128.27 90)
+			(effects
+				(font
+					(size 1.27 1.27)
+				)
+				(hide yes)
+			)
+		)
 		(pin "1"
 		)
@@
 		(unit 1)
 		(exclude_from_sim no)
-		(in_bom yes)
+		(in_bom no)
 		(on_board yes)
 		(dnp no)
@@
 		(unit 1)
 		(exclude_from_sim no)
-		(in_bom yes)
-		(on_board yes)
-		(dnp no)
+		(in_bom no)
+		(on_board yes)
+		(dnp no)

Commit message: board rc2
Parts:
- R5: value 1k -> 3k3; LCSC Part C11702 -> C25890
- R6: value 2k2 -> 100k; LCSC Part C25879 -> C25741
Connections:
- net GND: now also R5.2
- net at R4.2, R5.1, U5.4 (VSENSE): now also R6.1
Other:
- moved on the sheet: R5, R6
Changed lines of the file:
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@@
+	)
+	(junction
+		(at 147.32 69.85)
+		(diameter 0)
+		(color 0 0 0 0)
+	)
+	(junction
+		(at 147.32 59.69)
+		(diameter 0)
+		(color 0 0 0 0)
 	)
 	(junction
@@
 	(wire
 		(pts
+			(xy 147.32 69.85) (xy 147.32 71.12)
+		)
+		(stroke
+			(width 0)
+			(type default)
+		)
+	)
+	(wire
+		(pts
 			(xy 129.54 44.45) (xy 129.54 45.72)
 		)
@@
 	(wire
 		(pts
+			(xy 151.13 68.58) (xy 151.13 69.85)
+		)
+		(stroke
+			(width 0)
+			(type default)
+		)
+	)
+	(wire
+		(pts
+			(xy 147.32 59.69) (xy 143.51 59.69)
+		)
+		(stroke
+			(width 0)
+			(type default)
+		)
+	)
+	(wire
+		(pts
 			(xy 39.37 48.26) (xy 39.37 44.45)
 		)
@@
 	(wire
 		(pts
+			(xy 143.51 59.69) (xy 143.51 60.96)
+		)
+		(stroke
+			(width 0)
+			(type default)
+		)
+	)
+	(wire
+		(pts
 			(xy 64.77 44.45) (xy 64.77 45.72)
 		)
@@
 	(wire
 		(pts
+			(xy 143.51 69.85) (xy 143.51 68.58)
+		)
+		(stroke
+			(width 0)
+			(type default)
+		)
+	)
+	(wire
+		(pts
 			(xy 147.32 57.15) (xy 147.32 59.69)
 		)
@@
 	(wire
 		(pts
+			(xy 147.32 59.69) (xy 151.13 59.69)
+		)
+		(stroke
+			(width 0)
+			(type default)
+		)
+	)
+	(wire
+		(pts
+			(xy 151.13 59.69) (xy 151.13 60.96)
+		)
+		(stroke
+			(width 0)
+			(type default)
+		)
+	)
+	(wire
+		(pts
 			(xy 82.55 60.96) (xy 83.82 60.96)
 		)
@@
 		(pts
 			(xy 46.99 44.45) (xy 46.99 45.72)
+		)
+		(stroke
+			(width 0)
+			(type default)
+		)
+	)
+	(wire
+		(pts
+			(xy 147.32 69.85) (xy 151.13 69.85)
+		)
+		(stroke
+			(width 0)
+			(type default)
+		)
+	)
+	(wire
+		(pts
+			(xy 143.51 69.85) (xy 147.32 69.85)
 		)
 		(stroke
@@
 	(symbol
 		(lib_id "Device:R")
-		(at 147.32 63.5 0)
+		(at 143.51 64.77 0)
 		(unit 1)
 		(exclude_from_sim no)
@@
 		(dnp no)
 		(property "Reference" "R5"
-			(at 144.78 64.77 90)
-			(effects
-				(font
-					(size 1.27 1.27)
-				)
-				(justify left)
-			)
-		)
-		(property "Value" "1k"
-			(at 149.86 64.77 90)
+			(at 140.97 66.04 90)
+			(effects
+				(font
+					(size 1.27 1.27)
+				)
+				(justify left)
+			)
+		)
+		(property "Value" "3k3"
+			(at 146.05 66.04 90)
 			(effects
 				(font
@@
 		)
 		(property "Footprint" "Resistor_SMD:R_0402_1005Metric"
-			(at 145.542 63.5 90)
+			(at 141.732 64.77 90)
 			(effects
 				(font
@@
 		)
 		(property "Datasheet" "~"
-			(at 147.32 63.5 0)
+			(at 143.51 64.77 0)
 			(effects
 				(font
@@
 		)
 		(property "Description" "Resistor"
-			(at 147.32 63.5 0)
-			(effects
-				(font
-					(size 1.27 1.27)
-				)
-				(hide yes)
-			)
-		)
-		(property "LCSC Part" "C11702"
-			(at 147.32 63.5 0)
+			(at 143.51 64.77 0)
+			(effects
+				(font
+					(size 1.27 1.27)
+				)
+				(hide yes)
+			)
+		)
+		(property "LCSC Part" "C25890"
+			(at 143.51 64.77 0)
 			(effects
 				(font
@@
 		)
 		(property "JLCPCB BOM" ""
-			(at 147.32 63.5 0)
+			(at 143.51 64.77 0)
 			(effects
 				(font
@@
 	(symbol
 		(lib_id "power:GND")
-		(at 147.32 74.93 0)
+		(at 147.32 71.12 0)
 		(unit 1)
 		(exclude_from_sim no)
@@
 		(fields_autoplaced yes)
 		(property "Reference" "#PWR055"
-			(at 147.32 81.28 0)
+			(at 147.32 77.47 0)
 			(effects
 				(font
@@
 		)
 		(property "Value" "GND"
-			(at 147.32 80.01 0)
+			(at 147.32 76.2 0)
 			(effects
 				(font
@@
 		)
 		(property "Footprint" ""
-			(at 147.32 74.93 0)
+			(at 147.32 71.12 0)
 			(effects
 				(font
@@
 		)
 		(property "Datasheet" ""
-			(at 147.32 74.93 0)
+			(at 147.32 71.12 0)
 			(effects
 				(font
@@
 		)
 		(property "Description" "Power symbol creates a global label with name \"GND\" , ground"
-			(at 147.32 74.93 0)
+			(at 147.32 71.12 0)
 			(effects
 				(font
@@
 	(symbol
 		(lib_id "Device:R")
-		(at 147.32 71.12 0)
+		(at 151.13 64.77 0)
 		(unit 1)
 		(exclude_from_sim no)
@@
 		(dnp no)
 		(property "Reference" "R6"
-			(at 144.78 72.39 90)
-			(effects
-				(font
-					(size 1.27 1.27)
-				)
-				(justify left)
-			)
-		)
-		(property "Value" "2k2"
-			(at 149.86 72.39 90)
+			(at 148.59 66.04 90)
+			(effects
+				(font
+					(size 1.27 1.27)
+				)
+				(justify left)
+			)
+		)
+		(property "Value" "100k"
+			(at 153.67 66.04 90)
 			(effects
 				(font
@@
 		)
 		(property "Footprint" "Resistor_SMD:R_0402_1005Metric"
-			(at 145.542 71.12 90)
+			(at 149.352 64.77 90)
 			(effects
 				(font
@@
 		)
 		(property "Datasheet" "~"
-			(at 147.32 71.12 0)
+			(at 151.13 64.77 0)
 			(effects
 				(font
@@
 		)
 		(property "Description" "Resistor"
-			(at 147.32 71.12 0)
-			(effects
-				(font
-					(size 1.27 1.27)
-				)
-				(hide yes)
-			)
-		)
-		(property "LCSC Part" "C25879"
-			(at 147.32 71.12 0)
+			(at 151.13 64.77 0)
+			(effects
+				(font
+					(size 1.27 1.27)
+				)
+				(hide yes)
+			)
+		)
+		(property "LCSC Part" "C25741"
+			(at 151.13 64.77 0)
 			(effects
 				(font
@@
 		)
 		(property "JLCPCB BOM" ""
-			(at 147.32 71.12 0)
-			(effects
-				(font
+			(at 151.13 64.77 0)
+			(effects
+				(font
